File: hardware/kicad/STM32H743_DataLogger/Analog_Inputs.kicad_sch (KiCad schematic)
At the start: 11 parts, among them J20 AI_CH0 Input, J21 AI_CH1 Input, J22 AI_CH2 Input, J23 AI_CH3 Input, U20 OPA2376AIDGKR

Commit message: feat: Add P9E silkscreen branding, fix BOM/schematic cross-check issues
- Add complete silkscreen: P9E branding (3.5mm bold), company name,
  website, product info (Weather Station v2.0), functional area labels,
  connector pin labels, LED labels, compliance marks on back
- Fix BOM: add missing J12/J13/J14/R14-R16, resolve LED4 duplicate
  (renamed to LED5 for BLE), fix C101 conflict with C104
- Complete analog input schematic channels 1-3 (TVS, precision resistors,
  anti-alias RC filter, OPA2376 U21 for Ch2-3)
- Complete digital I/O schematic: add optocouplers U32-U37, current
  limiting resistors, pull-ups R38-R44 for DI Ch1-7, relays K2-K4
- Rebrand all files from SCADA Systems to P9E Microsystems Pvt Ltd
- Update revision to 2.0, date to 2026-03-20

https://claude.ai/code/session_01XsiZ6LJT6X46LKY8yEbRbx
Parts:
- added C61, C62, C63: 100nF C0G, Capacitor_SMD:C_0402_1005Metric, symbol Device:C
- added D11, D12, D13: PESD5V0S1BA, Diode_SMD:D_SOD-323, symbol Device:D_TVS
- added R24, R28, R32: 249R 0.1%, Resistor_SMD:R_0805_2012Metric, symbol Device:R
- added R25, R29, R33: 20k 0.1%, Resistor_SMD:R_0805_2012Metric, symbol Device:R
- added R26, R30x, R34: 10k 0.1%, Resistor_SMD:R_0805_2012Metric, symbol Device:R
- added R27, R31x, R35: 1k, Resistor_SMD:R_0402_1005Metric, symbol Device:R
- added U21: OPA2376AIDGKR, Package_SO:MSOP-8_3x3mm_P0.65mm, symbol Amplifier_Operational:OPA2376
Other:
- company: SCADA Systems -> P9E Microsystems Pvt Ltd
