File: hardware/kicad/STM32H743_DataLogger/Analog_Inputs.kicad_sch (KiCad schematic)
At the start: 30 parts, among them J20 AI_CH0 Input, J21 AI_CH1 Input, J22 AI_CH2 Input, J23 AI_CH3 Input, U20 OPA2376AIDGKR, U21 OPA2376AIDGKR

Commit message: Complete mfg PCB placement, fix designator conflicts, sync BOM
Manufacturing PCB (STM32H743_DataLogger_mfg.kicad_pcb):
- Add all missing multi-channel footprints: analog channels 1-3
  (D11-D13, R24-R35, C61-C63) plus second op-amp U21
- Add full 8-channel digital input chain (R100-R107 limiters,
  U30/U32-U38 optocouplers, R108-R115 pull-ups) with new
  DI_n_LED nets instead of floating net 0
- Add relays K2-K4 and replace the oversized SANYOU SRD placeholder
  with an HF46F-G/5-HS1T form-A footprint; wire relay contacts to
  J40-J43 via new DOn_NO / DOn_COM nets
- Add C104 (EEPROM decoupling), LED4 + R17 (comm activity indicator)
- Rename the BLE indicator from LED4 to LED5 to match the schematic
- Replace silkscreen branding with the full P9E block (company mark,
  P9E Microsystems Pvt Ltd, www.p9e.in, product, specs) on F.SilkS and
  P/N, S/N, compliance marks and origin on B.SilkS; www.p9e.io and the
  stale "SCADA Systems" text are gone
- Resolve all 26 footprint overlaps, pull the USB-C receptacle fully
  on-board, move fiducials clear of mounting holes, and drop the 22
  stitching vias that landed on pads

Schematics:
- Renumber Digital_IO resistors to R100-R115 and the eighth
  optocoupler to U38, removing the R31x/R40x placeholder designators
  and the R30/R31/R40/R41 collisions with Analog_Inputs and RS485_CAN
- Add C104 to Storage and LED4 + R17 to the MCU sheet

BOM: update the digital I/O and analog designator ranges to match,
add R17, correct the relay type to SPST-NO, and refresh the totals
(116 line items, 211 components).

Co-Authored-By: Claude Opus 5 <noreply@anthropic.com>
Claude-Session: https://claude.ai/code/session_01XsiZ6LJT6X46LKY8yEbRbx
Parts:
- renumbered R30x to R30, R31x to R31
Changed lines of the file:
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@@
     (exclude_from_sim no) (in_bom yes) (on_board yes) (dnp no)
     (uuid "AI-0034-R30")
-    (property "Reference" "R30x" (at 66.04 120.65 0) (effects (font (size 1.27 1.27))))
+    (property "Reference" "R30" (at 66.04 120.65 0) (effects (font (size 1.27 1.27))))
     (property "Value" "10k 0.1%" (at 63.5 123.19 0) (effects (font (size 1.27 1.27))))
     (property "Footprint" "Resistor_SMD:R_0805_2012Metric" (at 63.5 120.65 0) (effects (font (size 1.27 1.27)) hide))
@@
     (exclude_from_sim no) (in_bom yes) (on_board yes) (dnp no)
     (uuid "AI-0035-R31")
-    (property "Reference" "R31x" (at 78.74 114.3 0) (effects (font (size 1.27 1.27))))
+    (property "Reference" "R31" (at 78.74 114.3 0) (effects (font (size 1.27 1.27))))
     (property "Value" "1k" (at 76.2 116.84 0) (effects (font (size 1.27 1.27))))
     (property "Footprint" "Resistor_SMD:R_0402_1005Metric" (at 76.2 114.3 0) (effects (font (size 1.27 1.27)) hide))

Commit message: Verify every IC against its datasheet pinout; rebuild three, add missing parts
The MCU turned out not to be the only placeholder. With the symbol
libraries available I checked each IC's footprint wiring against the pin
names its datasheet-derived KiCad symbol gives — if a pin the datasheet
calls VDD is not on a supply net, the map was not derived from the
datasheet. Three ICs failed and are rebuilt:

- U50 W5500 had SPI on the Ethernet differential pins and supplies and
  grounds on ten wrong pads. Rebuilt from the 48-pin pinout: SPI on
  32-37, TX/RX pairs on 1/2/5/6, PMODE2..0 grounded for all-capable
  auto-negotiation.
- U40 ISO3082 had the receiver and driver swapped, the bus A/B pair one
  pin out, and GND2 carrying the isolated 5V supply.
- U1 TPS54560 had the switch node on pins 7 and 8, shorting SW to GND,
  and FB off pin 5.

Verifying the W5500 also showed three datasheet-required parts were never
placed: R56 (12.4k on EXRES1, sets transmit bias current), C87 (4.7uF on
TOCAP) and C88 (100nF on VBG). All three added.

Two ICs cannot be verified and are recorded as such rather than guessed
at. U60 is worse than a wiring error: the footprint is QFN-28 4x4mm on
0.4mm pitch, but SX1276IMLTRT is 6x6mm on 0.65mm pitch — the wrong
package outline entirely. U3's part is the DGN (MSOP-8-EP) variant and
the library only has KTT (TO-263-5), a different pinout, so it cannot
stand in. Six more ICs have no symbol at all and show the same sequential
pattern; they should be assumed wrong until checked.

Still open on the buck: EN, RT/CLK and COMP have no components on them.
RT/CLK sets the switching frequency and COMP is the compensation network,
so U1 will not regulate as drawn.

Also corrected twelve wrong schematic lib_ids against the real libraries;
35 of 44 now resolve, and the nine that need symbols drawn are listed in
docs/Schematic_Symbol_Audit.md.

BOM now 123 line items / 222 components; netlist 160 nets, all reaching
at least two pads.

Co-Authored-By: Claude O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
Parts:
- U20, U21: symbol Amplifier_Operational:OPA2376 -> Amplifier_Operational:OPA2376xxDGK
Changed lines of the file:
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@@
   )
   ;; Op-amp buffer (unity gain) - OPA2376 rail-to-rail, low offset
-  (symbol (lib_id "Amplifier_Operational:OPA2376") (at 107.95 50.8) (unit 1)
+  (symbol (lib_id "Amplifier_Operational:OPA2376xxDGK") (at 107.95 50.8) (unit 1)
     (exclude_from_sim no) (in_bom yes) (on_board yes) (dnp no)
     (uuid "AI-0010-U20")
@@
   )
   ;; U21 - Second OPA2376 serves Channels 2 & 3
-  (symbol (lib_id "Amplifier_Operational:OPA2376") (at 107.95 114.3) (unit 1)
+  (symbol (lib_id "Amplifier_Operational:OPA2376xxDGK") (at 107.95 114.3) (unit 1)
     (exclude_from_sim no) (in_bom yes) (on_board yes) (dnp no)
     (uuid "AI-0050-U21")
