File: hardware/kicad/STM32H743_DataLogger/Digital_IO.kicad_sch (KiCad schematic)
At the start: 17 parts, among them J30 DI_0, J31 DI_1, J32 DI_2, J33 DI_3, J34 DI_4, J35 DI_5, J36 DI_6, J37 DI_7, J40 DO_0 (NO/COM/NC), J41 DO_1 (NO/COM/NC)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

Commit message: feat: Add P9E silkscreen branding, fix BOM/schematic cross-check issues
- Add complete silkscreen: P9E branding (3.5mm bold), company name,
  website, product info (Weather Station v2.0), functional area labels,
  connector pin labels, LED labels, compliance marks on back
- Fix BOM: add missing J12/J13/J14/R14-R16, resolve LED4 duplicate
  (renamed to LED5 for BLE), fix C101 conflict with C104
- Complete analog input schematic channels 1-3 (TVS, precision resistors,
  anti-alias RC filter, OPA2376 U21 for Ch2-3)
- Complete digital I/O schematic: add optocouplers U32-U37, current
  limiting resistors, pull-ups R38-R44 for DI Ch1-7, relays K2-K4
- Rebrand all files from SCADA Systems to P9E Microsystems Pvt Ltd
- Update revision to 2.0, date to 2026-03-20

https://claude.ai/code/session_01XsiZ6LJT6X46LKY8yEbRbx
Parts:
- added K2, K3, K4: HF46F-G/5-HS1T, Relay_THT:Relay_SPDT_SANYOU_SRD_Series_Form_C, symbol Relay:SANYOU_SRD_Form_C
- added R31x, R32x, R33x, R34x, R35x, R36x, R37x: 4.7k, Resistor_SMD:R_0805_2012Metric, symbol Device:R
- added R38, R39, R40x, R41x, R42, R43, R44: 10k, Resistor_SMD:R_0402_1005Metric, symbol Device:R
- added U31x, U32, U33, U34, U35, U36, U37: TLP293(GR-TPL,E, Package_SO:SOP-4_3.8x4.1mm_P2.54mm, symbol Isolator:TLP293
Other:
- company: SCADA Systems -> P9E Microsystems Pvt Ltd
