File: hardware/kicad/STM32H743_DataLogger/Digital_IO.kicad_sch (KiCad schematic)
At the start: 41 parts, among them J30 DI_0, J31 DI_1, J32 DI_2, J33 DI_3, J34 DI_4, J35 DI_5, J36 DI_6, J37 DI_7, J40 DO_0 (NO/COM/NC), J41 DO_1 (NO/COM/NC), J42 DO_2 (NO/COM/NC), J43 DO_3 (NO/COM/NC), K1 HF46F-G/5-HS1T, K2 HF46F-G/5-HS1T, K3 HF46F-G/5-HS1T, K4 HF46F-G/5-HS1T, U30 TLP293(GR-TPL,E, U31 ULN2003AIDR, U31x TLP293(GR-TPL,E, U32 TLP293(GR-TPL,E, U33 TLP293(GR-TPL,E, U34 TLP293(GR-TPL,E, U35 TLP293(GR-TPL,E, U36 TLP293(GR-TPL,E, U37 TLP293(GR-TPL,E

Commit message: Complete mfg PCB placement, fix designator conflicts, sync BOM
Manufacturing PCB (STM32H743_DataLogger_mfg.kicad_pcb):
- Add all missing multi-channel footprints: analog channels 1-3
  (D11-D13, R24-R35, C61-C63) plus second op-amp U21
- Add full 8-channel digital input chain (R100-R107 limiters,
  U30/U32-U38 optocouplers, R108-R115 pull-ups) with new
  DI_n_LED nets instead of floating net 0
- Add relays K2-K4 and replace the oversized SANYOU SRD placeholder
  with an HF46F-G/5-HS1T form-A footprint; wire relay contacts to
  J40-J43 via new DOn_NO / DOn_COM nets
- Add C104 (EEPROM decoupling), LED4 + R17 (comm activity indicator)
- Rename the BLE indicator from LED4 to LED5 to match the schematic
- Replace silkscreen branding with the full P9E block (company mark,
  P9E Microsystems Pvt Ltd, www.p9e.in, product, specs) on F.SilkS and
  P/N, S/N, compliance marks and origin on B.SilkS; www.p9e.io and the
  stale "SCADA Systems" text are gone
- Resolve all 26 footprint overlaps, pull the USB-C receptacle fully
  on-board, move fiducials clear of mounting holes, and drop the 22
  stitching vias that landed on pads

Schematics:
- Renumber Digital_IO resistors to R100-R115 and the eighth
  optocoupler to U38, removing the R31x/R40x placeholder designators
  and the R30/R31/R40/R41 collisions with Analog_Inputs and RS485_CAN
- Add C104 to Storage and LED4 + R17 to the MCU sheet

BOM: update the digital I/O and analog designator ranges to match,
add R17, correct the relay type to SPST-NO, and refresh the totals
(116 line items, 211 components).

Co-Authored-By: Claude Opus 5 <noreply@anthropic.com>
Claude-Session: https://claude.ai/code/session_01XsiZ6LJT6X46LKY8yEbRbx
Parts:
- removed R31x, R32x, R33x, R34x, R35x, R36x, R37x: 4.7k, Resistor_SMD:R_0805_2012Metric, symbol Device:R
- removed R40x, R41x: 10k, Resistor_SMD:R_0402_1005Metric, symbol Device:R
- removed U31x: TLP293(GR-TPL,E, Package_SO:SOP-4_3.8x4.1mm_P2.54mm, symbol Isolator:TLP293
- added R101, R102, R103, R104, R105, R106, R107: 4.7k, Resistor_SMD:R_0805_2012Metric, symbol Device:R
- added R111, R112: 10k, Resistor_SMD:R_0402_1005Metric, symbol Device:R
- added U38: TLP293(GR-TPL,E, Package_SO:SOP-4_3.8x4.1mm_P2.54mm, symbol Isolator:TLP293
- renumbered R30 to R100, R31 to R108, R38 to R109, R39 to R110, R42 to R113, R43 to R114, R44 to R115
Changed lines of the file:
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@@
     (exclude_from_sim no) (in_bom yes) (on_board yes) (dnp no)
     (uuid "DIO-0002-R30")
-    (property "Reference" "R30" (at 40.64 44.45 0) (effects (font (size 1.27 1.27))))
+    (property "Reference" "R100" (at 40.64 44.45 0) (effects (font (size 1.27 1.27))))
     (property "Value" "4.7k" (at 38.1 46.99 0) (effects (font (size 1.27 1.27))))
     (property "Footprint" "Resistor_SMD:R_0805_2012Metric" (at 38.1 44.45 0) (effects (font (size 1.27 1.27)) hide))
@@
     (exclude_from_sim no) (in_bom yes) (on_board yes) (dnp no)
     (uuid "DIO-0004-R31")
-    (property "Reference" "R31" (at 72.39 38.1 0) (effects (font (size 1.27 1.27))))
+    (property "Reference" "R108" (at 72.39 38.1 0) (effects (font (size 1.27 1.27))))
     (property "Value" "10k" (at 69.85 40.64 0) (effects (font (size 1.27 1.27))))
     (property "Footprint" "Resistor_SMD:R_0402_1005Metric" (at 69.85 38.1 0) (effects (font (size 1.27 1.27)) hide))
@@
   (symbol (lib_id "Device:R") (at 38.1 57.15) (unit 1)
     (exclude_from_sim no) (in_bom yes) (on_board yes) (dnp no)
-    (uuid "DIO-0010-R31x")
-    (property "Reference" "R31x" (at 40.64 57.15 0) (effects (font (size 1.27 1.27))))
+    (uuid "DIO-0010-R101")
+    (property "Reference" "R101" (at 40.64 57.15 0) (effects (font (size 1.27 1.27))))
     (property "Value" "4.7k" (at 38.1 59.69 0) (effects (font (size 1.27 1.27))))
     (property "Footprint" "Resistor_SMD:R_0805_2012Metric" (at 38.1 57.15 0) (effects (font (size 1.27 1.27)) hide))
@@
   (symbol (lib_id "Isolator:TLP293") (at 57.15 57.15) (unit 1)
     (exclude_from_sim no) (in_bom yes) (on_board yes) (dnp no)
-    (uuid "DIO-0010-U31x")
-    (property "Reference" "U31x" (at 57.15 49.53 0) (effects (font (size 1.27 1.27))))
+    (uuid "DIO-0010-U38")
+    (property "Reference" "U38" (at 57.15 49.53 0) (effects (font (size 1.27 1.27))))
     (property "Value" "TLP293(GR-TPL,E" (at 57.15 52.07 0) (effects (font (size 1.27 1.27))))
     (property "Footprint" "Package_SO:SOP-4_3.8x4.1mm_P2.54mm" (at 57.15 57.15 0) (effects (font (size 1.27 1.27)) hide))
@@
     (exclude_from_sim no) (in_bom yes) (on_board yes) (dnp no)
     (uuid "DIO-0010-R38")
-    (property "Reference" "R38" (at 72.39 50.8 0) (effects (font (size 1.27 1.27))))
+    (property "Reference" "R109" (at 72.39 50.8 0) (effects (font (size 1.27 1.27))))
     (property "Value" "10k" (at 69.85 53.34 0) (effects (font (size 1.27 1.27))))
     (property "Footprint" "Resistor_SMD:R_0402_1005Metric" (at 69.85 50.8 0) (effects (font (size 1.27 1.27)) hide))
@@
   (symbol (lib_id "Device:R") (at 38.1 69.85) (unit 1)
     (exclude_from_sim no) (in_bom yes) (on_board yes) (dnp no)
-    (uuid "DIO-0011-R32x")
-    (property "Reference" "R32x" (at 40.64 69.85 0) (effects (font (size 1.27 1.27))))
+    (uuid "DIO-0011-R102")
+    (property "Reference" "R102" (at 40.64 69.85 0) (effects (font (size 1.27 1.27))))
     (property "Value" "4.7k" (at 38.1 72.39 0) (effects (font (size 1.27 1.27))))
     (property "Footprint" "Resistor_SMD:R_0805_2012Metric" (at 38.1 69.85 0) (effects (font (size 1.27 1.27)) hide))
@@
     (exclude_from_sim no) (in_bom yes) (on_board yes) (dnp no)
     (uuid "DIO-0011-R39")
-    (property "Reference" "R39" (at 72.39 63.5 0) (effects (font (size 1.27 1.27))))
+    (property "Reference" "R110" (at 72.39 63.5 0) (effects (font (size 1.27 1.27))))
     (property "Value" "10k" (at 69.85 66.04 0) (effects (font (size 1.27 1.27))))
     (property "Footprint" "Resistor_SMD:R_0402_1005Metric" (at 69.85 63.5 0) (effects (font (size 1.27 1.27)) hide))
@@
   (symbol (lib_id "Device:R") (at 38.1 82.55) (unit 1)
     (exclude_from_sim no) (in_bom yes) (on_board yes) (dnp no)
-    (uuid "DIO-0012-R33x")
-    (property "Reference" "R33x" (at 40.64 82.55 0) (effects (font (size 1.27 1.27))))
+    (uuid "DIO-0012-R103")
+    (property "Reference" "R103" (at 40.64 82.55 0) (effects (font (size 1.27 1.27))))
     (property "Value" "4.7k" (at 38.1 85.09 0) (effects (font (size 1.27 1.27))))
     (property "Footprint" "Resistor_SMD:R_0805_2012Metric" (at 38.1 82.55 0) (effects (font (size 1.27 1.27)) hide))
@@
   (symbol (lib_id "Device:R") (at 69.85 76.2) (unit 1)
     (exclude_from_sim no) (in_bom yes) (on_board yes) (dnp no)
-    (uuid "DIO-0012-R40x")
-    (property "Reference" "R40x" (at 72.39 76.2 0) (effects (font (size 1.27 1.27))))
+    (uuid "DIO-0012-R111")
+    (property "Reference" "R111" (at 72.39 76.2 0) (effects (font (size 1.27 1.27))))
     (property "Value" "10k" (at 69.85 78.74 0) (effects (font (size 1.27 1.27))))
     (property "Footprint" "Resistor_SMD:R_0402_1005Metric" (at 69.85 76.2 0) (effects (font (size 1.27 1.27)) hide))
@@
   (symbol (lib_id "Device:R") (at 38.1 95.25) (unit 1)
     (exclude_from_sim no) (in_bom yes) (on_board yes) (dnp no)
-    (uuid "DIO-0013-R34x")
-    (property "Reference" "R34x" (at 40.64 95.25 0) (effects (font (size 1.27 1.27))))
+    (uuid "DIO-0013-R104")
+    (property "Reference" "R104" (at 40.64 95.25 0) (effects (font (size 1.27 1.27))))
     (property "Value" "4.7k" (at 38.1 97.79 0) (effects (font (size 1.27 1.27))))
     (property "Footprint" "Resistor_SMD:R_0805_2012Metric" (at 38.1 95.25 0) (effects (font (size 1.27 1.27)) hide))
@@
   (symbol (lib_id "Device:R") (at 69.85 88.9) (unit 1)
     (exclude_from_sim no) (in_bom yes) (on_board yes) (dnp no)
-    (uuid "DIO-0013-R41x")
-    (property "Reference" "R41x" (at 72.39 88.9 0) (effects (font (size 1.27 1.27))))
+    (uuid "DIO-0013-R112")
+    (property "Reference" "R112" (at 72.39 88.9 0) (effects (font (size 1.27 1.27))))
     (property "Value" "10k" (at 69.85 91.44 0) (effects (font (size 1.27 1.27))))
     (property "Footprint" "Resistor_SMD:R_0402_1005Metric" (at 69.85 88.9 0) (effects (font (size 1.27 1.27)) hide))
@@
   (symbol (lib_id "Device:R") (at 38.1 107.95) (unit 1)
     (exclude_from_sim no) (in_bom yes) (on_board yes) (dnp no)
-    (uuid "DIO-0014-R35x")
-    (property "Reference" "R35x" (at 40.64 107.95 0) (effects (font (size 1.27 1.27))))
+    (uuid "DIO-0014-R105")
+    (property "Reference" "R105" (at 40.64 107.95 0) (effects (font (size 1.27 1.27))))
     (property "Value" "4.7k" (at 38.1 110.49 0) (effects (font (size 1.27 1.27))))
     (property "Footprint" "Resistor_SMD:R_0805_2012Metric" (at 38.1 107.95 0) (effects (font (size 1.27 1.27)) hide))
@@
     (exclude_from_sim no) (in_bom yes) (on_board yes) (dnp no)
     (uuid "DIO-0014-R42")
-    (property "Reference" "R42" (at 72.39 101.6 0) (effects (font (size 1.27 1.27))))
+    (property "Reference" "R113" (at 72.39 101.6 0) (effects (font (size 1.27 1.27))))
     (property "Value" "10k" (at 69.85 104.14 0) (effects (font (size 1.27 1.27))))
     (property "Footprint" "Resistor_SMD:R_0402_1005Metric" (at 69.85 101.6 0) (effects (font (size 1.27 1.27)) hide))
@@
   (symbol (lib_id "Device:R") (at 38.1 120.65) (unit 1)
     (exclude_from_sim no) (in_bom yes) (on_board yes) (dnp no)
-    (uuid "DIO-0015-R36x")
-    (property "Reference" "R36x" (at 40.64 120.65 0) (effects (font (size 1.27 1.27))))
+    (uuid "DIO-0015-R106")
+    (property "Reference" "R106" (at 40.64 120.65 0) (effects (font (size 1.27 1.27))))
     (property "Value" "4.7k" (at 38.1 123.19 0) (effects (font (size 1.27 1.27))))
     (property "Footprint" "Resistor_SMD:R_0805_2012Metric" (at 38.1 120.65 0) (effects (font (size 1.27 1.27)) hide))
@@
     (exclude_from_sim no) (in_bom yes) (on_board yes) (dnp no)
     (uuid "DIO-0015-R43")
-    (property "Reference" "R43" (at 72.39 114.3 0) (effects (font (size 1.27 1.27))))
+    (property "Reference" "R114" (at 72.39 114.3 0) (effects (font (size 1.27 1.27))))
     (property "Value" "10k" (at 69.85 116.84 0) (effects (font (size 1.27 1.27))))
     (property "Footprint" "Resistor_SMD:R_0402_1005Metric" (at 69.85 114.3 0) (effects (font (size 1.27 1.27)) hide))
@@
   (symbol (lib_id "Device:R") (at 38.1 133.35) (unit 1)
     (exclude_from_sim no) (in_bom yes) (on_board yes) (dnp no)
-    (uuid "DIO-0016-R37x")
-    (property "Reference" "R37x" (at 40.64 133.35 0) (effects (font (size 1.27 1.27))))
+    (uuid "DIO-0016-R107")
+    (property "Reference" "R107" (at 40.64 133.35 0) (effects (font (size 1.27 1.27))))
     (property "Value" "4.7k" (at 38.1 135.89 0) (effects (font (size 1.27 1.27))))
     (property "Footprint" "Resistor_SMD:R_0805_2012Metric" (at 38.1 133.35 0) (effects (font (size 1.27 1.27)) hide))
@@
     (exclude_from_sim no) (in_bom yes) (on_board yes) (dnp no)
     (uuid "DIO-0016-R44")
-    (property "Reference" "R44" (at 72.39 127 0) (effects (font (size 1.27 1.27))))
+    (property "Reference" "R115" (at 72.39 127 0) (effects (font (size 1.27 1.27))))
     (property "Value" "10k" (at 69.85 129.54 0) (effects (font (size 1.27 1.27))))
     (property "Footprint" "Resistor_SMD:R_0402_1005Metric" (at 69.85 127 0) (effects (font (size 1.27 1.27)) hide))

Commit message: Verify every IC against its datasheet pinout; rebuild three, add missing parts
The MCU turned out not to be the only placeholder. With the symbol
libraries available I checked each IC's footprint wiring against the pin
names its datasheet-derived KiCad symbol gives — if a pin the datasheet
calls VDD is not on a supply net, the map was not derived from the
datasheet. Three ICs failed and are rebuilt:

- U50 W5500 had SPI on the Ethernet differential pins and supplies and
  grounds on ten wrong pads. Rebuilt from the 48-pin pinout: SPI on
  32-37, TX/RX pairs on 1/2/5/6, PMODE2..0 grounded for all-capable
  auto-negotiation.
- U40 ISO3082 had the receiver and driver swapped, the bus A/B pair one
  pin out, and GND2 carrying the isolated 5V supply.
- U1 TPS54560 had the switch node on pins 7 and 8, shorting SW to GND,
  and FB off pin 5.

Verifying the W5500 also showed three datasheet-required parts were never
placed: R56 (12.4k on EXRES1, sets transmit bias current), C87 (4.7uF on
TOCAP) and C88 (100nF on VBG). All three added.

Two ICs cannot be verified and are recorded as such rather than guessed
at. U60 is worse than a wiring error: the footprint is QFN-28 4x4mm on
0.4mm pitch, but SX1276IMLTRT is 6x6mm on 0.65mm pitch — the wrong
package outline entirely. U3's part is the DGN (MSOP-8-EP) variant and
the library only has KTT (TO-263-5), a different pinout, so it cannot
stand in. Six more ICs have no symbol at all and show the same sequential
pattern; they should be assumed wrong until checked.

Still open on the buck: EN, RT/CLK and COMP have no components on them.
RT/CLK sets the switching frequency and COMP is the compensation network,
so U1 will not regulate as drawn.

Also corrected twelve wrong schematic lib_ids against the real libraries;
35 of 44 now resolve, and the nine that need symbols drawn are listed in
docs/Schematic_Symbol_Audit.md.

BOM now 123 line items / 222 components; netlist 160 nets, all reaching
at least two pads.

Co-Authored-By: Claude O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
Parts:
- U31: symbol Driver_Motor:ULN2003 -> Transistor_Array:ULN2003A
Changed lines of the file:
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@@
   ;; ============================================================
   ;; ULN2003 Darlington Driver Array
-  (symbol (lib_id "Driver_Motor:ULN2003") (at 152.4 69.85) (unit 1)
+  (symbol (lib_id "Transistor_Array:ULN2003A") (at 152.4 69.85) (unit 1)
     (exclude_from_sim no) (in_bom yes) (on_board yes) (dnp no)
     (uuid "DIO-0050-U31")
