File: hardware/kicad/STM32H743_DataLogger/Ethernet.kicad_sch (KiCad schematic)
At the start: 9 parts, among them J60 J0011D21BNL, U50 LAN8742A-CZ-TR

Commit message: feat: Upgrade to full industrial-grade components and SPI architecture
Major design changes for PLC-grade reliability:

Component Upgrades:
- Replace ESP32-C3 dual-MCU with ATWINC1500 WiFi (SPI2) + RN4870 BLE (UART7)
  Eliminates second processor, both rated -40 to +85°C industrial
- Replace LAN8742A RMII PHY with W5500 SPI Ethernet controller
  Hardwired TCP/IP stack, frees 11 RMII pins, simpler firmware
- Replace RFM95W module with SX1276IMLTRT bare IC (-40 to +85°C)
  Full industrial temp range with 32MHz TCXO and custom RF matching
- Add TPS3823-33 external hardware watchdog (1.6s timeout)

Industrial Compliance:
- All key ICs rated -40 to +85°C (industrial grade)
- HumiSeal 1B73 conformal coating spec (MIL-I-46058C)
- EMC compliance targets: IEC 61000-4-2/4/5/6/8
- Ferrite beads on Ethernet pairs for EMI

Architecture: Single MCU (STM32H743) with all peripherals as SPI/UART slaves
- SPI1: SX1276 LoRa
- SPI2: ATWINC1500 WiFi
- SPI3: W25Q64JV Flash
- SPI4: W5500 Ethernet
- UART4: SIM7600G-H GSM/LTE
- UART7: RN4870 BLE

Updated BOM: ~170 components, ~$142/unit (1pc), ~$90/unit (100pc)

https://claude.ai/code/session_01XsiZ6LJT6X46LKY8yEbRbx
Parts:
- removed R50, R51: 49.9R, Resistor_SMD:R_0402_1005Metric, symbol Device:R
- removed R52: 10k, Resistor_SMD:R_0402_1005Metric, symbol Device:R
- added C82B, C85: 10uF, Capacitor_SMD:C_0805_2012Metric, symbol Device:C
- added C83, C84: 18pF, Capacitor_SMD:C_0402_1005Metric, symbol Device:C
- added C86: 100nF, Capacitor_SMD:C_0402_1005Metric, symbol Device:C
- added FB1, FB2, FB3, FB4: BLM18PG121SN1D, Inductor_SMD:L_0603_1608Metric, symbol Device:Ferrite_Bead
- added R53, R54, R55: 10k, Resistor_SMD:R_0402_1005Metric, symbol Device:R
- added Y3: 25MHz, Crystal:Crystal_SMD_3215-4Pin_3.2x1.5mm, symbol Device:Crystal
- C82: value 10uF -> 100nF; footprint Capacitor_SMD:C_0805_2012Metric -> Capacitor_SMD:C_0402_1005Metric; MPN GRM21BR61A106ME51L -> GRM155R71C104KA88D
- U50: value LAN8742A-CZ-TR -> W5500; footprint Package_DFN_QFN:QFN-24-1EP_4x4mm_P0.5mm_EP2.6x2.6mm -> Package_DFN_QFN:QFN-48-1EP_7x7mm_P0.5mm_EP5.6x5.6mm; symbol Interface_Ethernet:LAN8742A-CZ-TR -> Interface_Ethernet:W5500; MPN LAN8742A-CZ-TR -> W5500; Manufacturer Microchip -> WIZnet
Other:
- note added: "ETHERNET 10/100 DESIGN (Rev 1.1 - W5500) Controller: W5500 (WIZnet) - QFN-48 - Hardwired TCP/IP stack (no lwIP needed!) - Integrated 10/100 MAC + PHY - SPI interface up to 80MHz (SPI4 on STM32) - 8 simultaneous hardware sockets - 32KB internal TX/RX buffer - Industrial temp: -40 to +85C - Own 25MHz crystal (independent of MCU HSE) Advantages over LAN8742A (PHY-only): - Only 4 SPI pins vs 11 RMII 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"
- note removed: "ETHERNET 10/100 DESIGN PHY: LAN8742A-CZ-TR (QFN-24) - RMII interface to STM32H743 - 25MHz REF_CLK from HSE crystal - Internal 1.2V regulator - Auto-MDIX support - IEEE 802.3 / 802.3u compliant Magnetics: J0011D21BNL (RJ45 + integrated magnetics) - 10/100 Base-TX - Link/Activity LEDs integrated - Shielded connector ESD: PESD5V0S2BT on all data lines Termination: 49.9R series on TX+/TX-"
- title: Ethernet 10/100 - LAN8742A RMII PHY -> Ethernet 10/100 - W5500 SPI Ethernet Controller

Commit message: feat: Add P9E silkscreen branding, fix BOM/schematic cross-check issues
- Add complete silkscreen: P9E branding (3.5mm bold), company name,
  website, product info (Weather Station v2.0), functional area labels,
  connector pin labels, LED labels, compliance marks on back
- Fix BOM: add missing J12/J13/J14/R14-R16, resolve LED4 duplicate
  (renamed to LED5 for BLE), fix C101 conflict with C104
- Complete analog input schematic channels 1-3 (TVS, precision resistors,
  anti-alias RC filter, OPA2376 U21 for Ch2-3)
- Complete digital I/O schematic: add optocouplers U32-U37, current
  limiting resistors, pull-ups R38-R44 for DI Ch1-7, relays K2-K4
- Rebrand all files from SCADA Systems to P9E Microsystems Pvt Ltd
- Update revision to 2.0, date to 2026-03-20

https://claude.ai/code/session_01XsiZ6LJT6X46LKY8yEbRbx
Other:
- company: SCADA Systems -> P9E Microsystems Pvt Ltd
Changed lines of the file:
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@@
     (date "2026-03-15")
     (rev "1.1")
-    (company "SCADA Systems")
+    (company "P9E Microsystems Pvt Ltd")
     (comment 1 "W5500 Hardwired TCP/IP + MAC + PHY, SPI interface")
     (comment 2 "RJ45 with integrated magnetics and LEDs")
