File: hardware/kicad/STM32H743_DataLogger/Ethernet.kicad_sch (KiCad schematic)
At the start: 19 parts, among them J60 J0011D21BNL, U50 W5500, Y3 25MHz

Commit message: Verify every IC against its datasheet pinout; rebuild three, add missing parts
The MCU turned out not to be the only placeholder. With the symbol
libraries available I checked each IC's footprint wiring against the pin
names its datasheet-derived KiCad symbol gives — if a pin the datasheet
calls VDD is not on a supply net, the map was not derived from the
datasheet. Three ICs failed and are rebuilt:

- U50 W5500 had SPI on the Ethernet differential pins and supplies and
  grounds on ten wrong pads. Rebuilt from the 48-pin pinout: SPI on
  32-37, TX/RX pairs on 1/2/5/6, PMODE2..0 grounded for all-capable
  auto-negotiation.
- U40 ISO3082 had the receiver and driver swapped, the bus A/B pair one
  pin out, and GND2 carrying the isolated 5V supply.
- U1 TPS54560 had the switch node on pins 7 and 8, shorting SW to GND,
  and FB off pin 5.

Verifying the W5500 also showed three datasheet-required parts were never
placed: R56 (12.4k on EXRES1, sets transmit bias current), C87 (4.7uF on
TOCAP) and C88 (100nF on VBG). All three added.

Two ICs cannot be verified and are recorded as such rather than guessed
at. U60 is worse than a wiring error: the footprint is QFN-28 4x4mm on
0.4mm pitch, but SX1276IMLTRT is 6x6mm on 0.65mm pitch — the wrong
package outline entirely. U3's part is the DGN (MSOP-8-EP) variant and
the library only has KTT (TO-263-5), a different pinout, so it cannot
stand in. Six more ICs have no symbol at all and show the same sequential
pattern; they should be assumed wrong until checked.

Still open on the buck: EN, RT/CLK and COMP have no components on them.
RT/CLK sets the switching frequency and COMP is the compensation network,
so U1 will not regulate as drawn.

Also corrected twelve wrong schematic lib_ids against the real libraries;
35 of 44 now resolve, and the nine that need symbols drawn are listed in
docs/Schematic_Symbol_Audit.md.

BOM now 123 line items / 222 components; netlist 160 nets, all reaching
at least two pads.

Co-Authored-By: Claude O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
Parts:
- FB1, FB2, FB3, FB4: symbol Device:Ferrite_Bead -> Device:FerriteBead
Changed lines of the file:
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@@
   ;; TX PAIR FERRITE BEADS (EMI suppression per W5500 reference design)
   ;; ============================================================
-  (symbol (lib_id "Device:Ferrite_Bead") (at 139.7 82.55) (unit 1)
+  (symbol (lib_id "Device:FerriteBead") (at 139.7 82.55) (unit 1)
     (exclude_from_sim no) (in_bom yes) (on_board yes) (dnp no)
     (uuid "ETH-0011-FB1")
@@
     (property "Manufacturer" "Murata" (at 139.7 82.55 0) (effects (font (size 1.27 1.27)) hide))
   )
-  (symbol (lib_id "Device:Ferrite_Bead") (at 139.7 88.9) (unit 1)
+  (symbol (lib_id "Device:FerriteBead") (at 139.7 88.9) (unit 1)
     (exclude_from_sim no) (in_bom yes) (on_board yes) (dnp no)
     (uuid "ETH-0012-FB2")
@@
     (property "Manufacturer" "Murata" (at 139.7 88.9 0) (effects (font (size 1.27 1.27)) hide))
   )
-  (symbol (lib_id "Device:Ferrite_Bead") (at 139.7 95.25) (unit 1)
+  (symbol (lib_id "Device:FerriteBead") (at 139.7 95.25) (unit 1)
     (exclude_from_sim no) (in_bom yes) (on_board yes) (dnp no)
     (uuid "ETH-0013-FB3")
@@
     (property "Manufacturer" "Murata" (at 139.7 95.25 0) (effects (font (size 1.27 1.27)) hide))
   )
-  (symbol (lib_id "Device:Ferrite_Bead") (at 139.7 101.6) (unit 1)
+  (symbol (lib_id "Device:FerriteBead") (at 139.7 101.6) (unit 1)
     (exclude_from_sim no) (in_bom yes) (on_board yes) (dnp no)
     (uuid "ETH-0014-FB4")

Commit message: Add R56, C87 and C88 to the Ethernet sheet
The three W5500 support parts were placed on the board and added to the
BOM but not to the schematic, so the reference sets disagreed. Every
reference now appears in all three (mounting holes and fiducials aside,
which have no schematic symbol by design).

Co-Authored-By: Claude Opus 5 <noreply@anthropic.com>
Claude-Session: https://claude.ai/code/session_01XsiZ6LJT6X46LKY8yEbRbx
Parts:
- added C87: 4.7uF, Capacitor_SMD:C_0805_2012Metric, symbol Device:C
- added C88: 100nF, Capacitor_SMD:C_0402_1005Metric, symbol Device:C
- added R56: 12.4k 1%, Resistor_SMD:R_0402_1005Metric, symbol Device:R
Changed lines of the file:
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@@
     (uuid "ETH-TEXT-0001")
   )
+  ;; W5500 support required by the datasheet
+  (symbol (lib_id "Device:R") (at 190.5 165.1) (unit 1)
+    (exclude_from_sim no) (in_bom yes) (on_board yes) (dnp no)
+    (uuid "ETH-0060-R56")
+    (property "Reference" "R56" (at 193.04 165.1 0) (effects (font (size 1.27 1.27))))
+    (property "Value" "12.4k 1%" (at 190.5 167.64 0) (effects (font (size 1.27 1.27))))
+    (property "Footprint" "Resistor_SMD:R_0402_1005Metric" (at 190.5 165.1 0) (effects (font (size 1.27 1.27)) hide))
+    (property "MPN" "RC0402FR-0712K4L" (at 190.5 165.1 0) (effects (font (size 1.27 1.27)) hide))
+    (property "Description" "EXRES1 bias resistor - sets the PHY transmit current" (at 190.5 165.1 0) (effects (font (size 1.27 1.27)) hide))
+  )
+  (symbol (lib_id "Device:C") (at 203.2 165.1) (unit 1)
+    (exclude_from_sim no) (in_bom yes) (on_board yes) (dnp no)
+    (uuid "ETH-0061-C87")
+    (property "Reference" "C87" (at 205.74 163.83 0) (effects (font (size 1.27 1.27))))
+    (property "Value" "4.7uF" (at 203.2 167.64 0) (effects (font (size 1.27 1.27))))
+    (property "Footprint" "Capacitor_SMD:C_0805_2012Metric" (at 203.2 165.1 0) (effects (font (size 1.27 1.27)) hide))
+    (property "MPN" "GRM21BR61A475KA73L" (at 203.2 165.1 0) (effects (font (size 1.27 1.27)) hide))
+    (property "Description" "TOCAP - internal 1.2V transceiver regulator decoupling" (at 203.2 165.1 0) (effects (font (size 1.27 1.27)) hide))
+  )
+  (symbol (lib_id "Device:C") (at 215.9 165.1) (unit 1)
+    (exclude_from_sim no) (in_bom yes) (on_board yes) (dnp no)
+    (uuid "ETH-0062-C88")
+    (property "Reference" "C88" (at 218.44 163.83 0) (effects (font (size 1.27 1.27))))
+    (property "Value" "100nF" (at 215.9 167.64 0) (effects (font (size 1.27 1.27))))
+    (property "Footprint" "Capacitor_SMD:C_0402_1005Metric" (at 215.9 165.1 0) (effects (font (size 1.27 1.27)) hide))
+    (property "MPN" "GRM155R71C104KA88D" (at 215.9 165.1 0) (effects (font (size 1.27 1.27)) hide))
+    (property "Description" "VBG - bandgap reference decoupling" (at 215.9 165.1 0) (effects (font (size 1.27 1.27)) hide))
+  )
 )
