File: hardware/kicad/STM32H743_DataLogger/Power_Supply.kicad_sch (KiCad schematic)
At the start: 20 parts, among them J1 24VDC Input, Q1 SI4435DDY, U1 TPS54560DDAR, U2 TLV1117LV33DCYR, U3 TPS7A4533DGNR

Commit message: Close six unconnected nets found while exporting the netlist
Exporting the board to Specctra for routing surfaced six nets with only
one pad on them — they had nothing to connect to:

- VBUCK_BST reached only U1 pin 1. The buck had no bootstrap capacitor,
  so the high-side switch could never turn on and the 24V-to-5V stage
  would not start. Added C11 (100nF) from BST to the SW node.
- USART1_TX_BUF and USART1_RX_BUF dead-ended at R14/R15. J12 tapped the
  MCU side of the 33R series resistors, so the debug header was wired
  straight to the MCU and the resistors sat in mid-air. J12 now taps the
  buffered side, putting them in circuit as intended.
- GSM_DTR, GSM_RI and LORA_DIO1 reached only their module pins. The MCU
  has no spare pad (all 100 are assigned), so DTR gets a 10k pull-down
  (R18) to hold the modem out of sleep rather than floating, and RI and
  DIO1 come out to probe pads TP9/TP10.

Also added TP1-TP8 to the schematics; they existed only as PCB pads, so
the netlist and the board disagreed about them.

BOM now 120 line items / 219 components. Placement re-verified: 227
footprints, zero courtyard collisions, nothing off-board.

Co-Authored-By: Claude Opus 5 <noreply@anthropic.com>
Claude-Session: https://claude.ai/code/session_01XsiZ6LJT6X46LKY8yEbRbx
Parts:
- added C11: 100nF, Capacitor_SMD:C_0402_1005Metric, symbol Device:C
- added TP1: +3V3, TestPoint:TestPoint_Pad_1.0x1.0mm, symbol Connector:TestPoint
- added TP2: +5V, TestPoint:TestPoint_Pad_1.0x1.0mm, symbol Connector:TestPoint
- added TP3: +3V3A, TestPoint:TestPoint_Pad_1.0x1.0mm, symbol Connector:TestPoint
- added TP4: GND, TestPoint:TestPoint_Pad_1.0x1.0mm, symbol Connector:TestPoint
Changed lines of the file:
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@@
     (uuid "PS-TEXT-0001")
   )
+  ;; C11 - buck bootstrap capacitor (BST to SW).  Without it U1 cannot switch.
+  (symbol (lib_id "Device:C") (at 190.5 88.9) (unit 1)
+    (exclude_from_sim no) (in_bom yes) (on_board yes) (dnp no)
+    (uuid "PS-0040-C11")
+    (property "Reference" "C11" (at 193.04 87.63 0) (effects (font (size 1.27 1.27))))
+    (property "Value" "100nF" (at 190.5 91.44 0) (effects (font (size 1.27 1.27))))
+    (property "Footprint" "Capacitor_SMD:C_0402_1005Metric" (at 190.5 88.9 0) (effects (font (size 1.27 1.27)) hide))
+    (property "MPN" "GRM155R71C104KA88D" (at 190.5 88.9 0) (effects (font (size 1.27 1.27)) hide))
+    (property "Manufacturer" "Murata" (at 190.5 88.9 0) (effects (font (size 1.27 1.27)) hide))
+  )
+  ;; Probe test points
+  (symbol (lib_id "Connector:TestPoint") (at 165.1 190.5) (unit 1)
+    (exclude_from_sim no) (in_bom yes) (on_board yes) (dnp no)
+    (uuid "PS-0041-TP1")
+    (property "Reference" "TP1" (at 165.1 186.69 0) (effects (font (size 1.27 1.27))))
+    (property "Value" "+3V3" (at 165.1 189.23 0) (effects (font (size 1.27 1.27))))
+    (property "Footprint" "TestPoint:TestPoint_Pad_1.0x1.0mm" (at 165.1 190.5 0) (effects (font (size 1.27 1.27)) hide))
+  )
+  (symbol (lib_id "Connector:TestPoint") (at 177.8 190.5) (unit 1)
+    (exclude_from_sim no) (in_bom yes) (on_board yes) (dnp no)
+    (uuid "PS-0042-TP2")
+    (property "Reference" "TP2" (at 177.8 186.69 0) (effects (font (size 1.27 1.27))))
+    (property "Value" "+5V" (at 177.8 189.23 0) (effects (font (size 1.27 1.27))))
+    (property "Footprint" "TestPoint:TestPoint_Pad_1.0x1.0mm" (at 177.8 190.5 0) (effects (font (size 1.27 1.27)) hide))
+  )
+  (symbol (lib_id "Connector:TestPoint") (at 190.5 190.5) (unit 1)
+    (exclude_from_sim no) (in_bom yes) (on_board yes) (dnp no)
+    (uuid "PS-0043-TP3")
+    (property "Reference" "TP3" (at 190.5 186.69 0) (effects (font (size 1.27 1.27))))
+    (property "Value" "+3V3A" (at 190.5 189.23 0) (effects (font (size 1.27 1.27))))
+    (property "Footprint" "TestPoint:TestPoint_Pad_1.0x1.0mm" (at 190.5 190.5 0) (effects (font (size 1.27 1.27)) hide))
+  )
+  (symbol (lib_id "Connector:TestPoint") (at 203.2 190.5) (unit 1)
+    (exclude_from_sim no) (in_bom yes) (on_board yes) (dnp no)
+    (uuid "PS-0044-TP4")
+    (property "Reference" "TP4" (at 203.2 186.69 0) (effects (font (size 1.27 1.27))))
+    (property "Value" "GND" (at 203.2 189.23 0) (effects (font (size 1.27 1.27))))
+    (property "Footprint" "TestPoint:TestPoint_Pad_1.0x1.0mm" (at 203.2 190.5 0) (effects (font (size 1.27 1.27)) hide))
+  )
 )

Commit message: Verify every IC against its datasheet pinout; rebuild three, add missing parts
The MCU turned out not to be the only placeholder. With the symbol
libraries available I checked each IC's footprint wiring against the pin
names its datasheet-derived KiCad symbol gives — if a pin the datasheet
calls VDD is not on a supply net, the map was not derived from the
datasheet. Three ICs failed and are rebuilt:

- U50 W5500 had SPI on the Ethernet differential pins and supplies and
  grounds on ten wrong pads. Rebuilt from the 48-pin pinout: SPI on
  32-37, TX/RX pairs on 1/2/5/6, PMODE2..0 grounded for all-capable
  auto-negotiation.
- U40 ISO3082 had the receiver and driver swapped, the bus A/B pair one
  pin out, and GND2 carrying the isolated 5V supply.
- U1 TPS54560 had the switch node on pins 7 and 8, shorting SW to GND,
  and FB off pin 5.

Verifying the W5500 also showed three datasheet-required parts were never
placed: R56 (12.4k on EXRES1, sets transmit bias current), C87 (4.7uF on
TOCAP) and C88 (100nF on VBG). All three added.

Two ICs cannot be verified and are recorded as such rather than guessed
at. U60 is worse than a wiring error: the footprint is QFN-28 4x4mm on
0.4mm pitch, but SX1276IMLTRT is 6x6mm on 0.65mm pitch — the wrong
package outline entirely. U3's part is the DGN (MSOP-8-EP) variant and
the library only has KTT (TO-263-5), a different pinout, so it cannot
stand in. Six more ICs have no symbol at all and show the same sequential
pattern; they should be assumed wrong until checked.

Still open on the buck: EN, RT/CLK and COMP have no components on them.
RT/CLK sets the switching frequency and COMP is the compensation network,
so U1 will not regulate as drawn.

Also corrected twelve wrong schematic lib_ids against the real libraries;
35 of 44 now resolve, and the nine that need symbols drawn are listed in
docs/Schematic_Symbol_Audit.md.

BOM now 123 line items / 222 components; netlist 160 nets, all reaching
at least two pads.

Co-Authored-By: Claude O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
Parts:
- L1: symbol Device:L_Core_Ferrite -> Device:L_Ferrite
- Q1: symbol Device:Q_PMOS_GSD -> Transistor_FET:Q_PMOS_GSD
- U1: symbol Regulator_Switching:TPS54560 -> Regulator_Switching:TPS54560BDDA
- U3: symbol Regulator_Linear:TPS7A4533 -> Regulator_Linear:TPS7A4533DGN
Changed lines of the file:
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@@
   ;; D2 - Reverse polarity protection MOSFET
   (symbol
-    (lib_id "Device:Q_PMOS_GSD")
+    (lib_id "Transistor_FET:Q_PMOS_GSD")
     (at 50.8 44.45)
     (unit 1)
@@
   ;; L1 - Common mode choke for EMI filtering
   (symbol
-    (lib_id "Device:L_Core_Ferrite")
+    (lib_id "Device:L_Ferrite")
     (at 63.5 44.45)
     (unit 1)
@@
   ;; ============================================================
   (symbol
-    (lib_id "Regulator_Switching:TPS54560")
+    (lib_id "Regulator_Switching:TPS54560BDDA")
     (at 101.6 57.15)
     (unit 1)
@@
   ;; ============================================================
   (symbol
-    (lib_id "Regulator_Linear:TPS7A4533")
+    (lib_id "Regulator_Linear:TPS7A4533DGN")
     (at 177.8 82.55)
     (unit 1)
