File: hardware/kicad/STM32H743_DataLogger/RS485_CAN.kicad_sch (KiCad schematic)
At the start: 9 parts, among them J50 RS485 (A/B/GND), J51 CAN (H/L/GND), U40 ISO3082DWR, U41 ISO1042BQDWRQ1

Commit message: feat: Add P9E silkscreen branding, fix BOM/schematic cross-check issues
- Add complete silkscreen: P9E branding (3.5mm bold), company name,
  website, product info (Weather Station v2.0), functional area labels,
  connector pin labels, LED labels, compliance marks on back
- Fix BOM: add missing J12/J13/J14/R14-R16, resolve LED4 duplicate
  (renamed to LED5 for BLE), fix C101 conflict with C104
- Complete analog input schematic channels 1-3 (TVS, precision resistors,
  anti-alias RC filter, OPA2376 U21 for Ch2-3)
- Complete digital I/O schematic: add optocouplers U32-U37, current
  limiting resistors, pull-ups R38-R44 for DI Ch1-7, relays K2-K4
- Rebrand all files from SCADA Systems to P9E Microsystems Pvt Ltd
- Update revision to 2.0, date to 2026-03-20

https://claude.ai/code/session_01XsiZ6LJT6X46LKY8yEbRbx
Other:
- company: SCADA Systems -> P9E Microsystems Pvt Ltd
Changed lines of the file:
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@@
     (date "2026-03-15")
     (rev "1.0")
-    (company "SCADA Systems")
+    (company "P9E Microsystems Pvt Ltd")
     (comment 1 "Isolated RS485 (ISO3082) + Isolated CAN FD (ISO1042)")
     (comment 2 "Industrial fieldbus connectivity")
