File: hardware/kicad/STM32H743_DataLogger/RS485_CAN.kicad_sch (KiCad schematic)
At the start: 9 parts, among them J50 RS485 (A/B/GND), J51 CAN (H/L/GND), U40 ISO3082DWR, U41 ISO1042BQDWRQ1

Commit message: Re-floorplan mfg PCB on real courtyards; make the isolation real
Footprints carried pads only, so collision checks were meaningless — a
10x9.6mm terminal block measured as 2.4mm. Every footprint now has an
F.CrtYd body rect (package body union pad extents), which exposed 74
courtyard collisions the old pad-only check called clean, including
terminal blocks stacked at 4mm pitch and the 30x30mm SIM7600 sitting on
top of six neighbours.

Placement is now generated by an explicit floorplan rather than nudged:
- Field wiring lives on the two long edges. Bottom: 24VDC in, the four
  analog inputs, then the four relay outputs. Top: RS485 and CAN behind
  the isolation barrier, then the eight digital inputs.
- RJ45, USB-C and the three SMA antennas moved to the right edge;
  microSD to the left.
- Each circuit block is packed into a region adjacent to its own
  connector (analog over its terminals, relays over theirs, W5500
  beside the RJ45, and so on), at 33-65% area fill.
- Result: 223 footprints, zero courtyard collisions, nothing off-board.

Two isolation defects found and fixed:
- ISO3082 and ISO1042 had no isolated bus-side supply at all —
  RS485_ISO_VCC and CAN_ISO_VCC were undriven, so the 5kVrms parts could
  not work. Added U42/U43 (NXJ1S0505MC-R13, 5.2kVDC 1W) and C71-C74.
- The optocoupled digital inputs were not isolated: every TLP293 LED
  cathode and every field terminal's second pin sat on logic GND, making
  the field wiring and logic ground one node. Added a floating DI_COM
  field return and moved both onto it.

Isolation is now built into the copper: the GND and +3V3 pours are
notched away from the top-left corner, the RS485 and CAN field sides get
their own floating pours (8mm to main copper on the outside, 4mm between
the two domains), milled slots run under U40-U43 where they cross the
barrier, and a copper keepout on all four layers stops any layer
bridging the optocoupler row. Verified: no logic-net pad lies inside the
isolated pocket. The isolato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
Parts:
- added C71, C72, C73, C74: 10uF, Capacitor_SMD:C_0805_2012Metric, symbol Device:C
- added U42, U43: NXJ1S0505MC-R13, Converter_DCDC:Converter_DCDC_NXJ1S_SMD, symbol Converter_DCDC:NXJ1S0505MC-R13
Changed lines of the file:
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@@
+  )
+  ;; ============================================================
+  ;; ISOLATED BUS-SIDE SUPPLIES
+  ;; The ISO3082 / ISO1042 bus sides need their own floating 5V rail; without
+  ;; these converters RS485_ISO_VCC / CAN_ISO_VCC are undriven and the galvanic
+  ;; isolation is defeated.  NXJ1S is rated 5.2kVDC to match the transceivers.
+  ;; ============================================================
+  (symbol (lib_id "Converter_DCDC:NXJ1S0505MC-R13") (at 69.85 165.1) (unit 1)
+    (exclude_from_sim no) (in_bom yes) (on_board yes) (dnp no)
+    (uuid "COM-0014-U42")
+    (property "Reference" "U42" (at 69.85 157.48 0) (effects (font (size 1.27 1.27))))
+    (property "Value" "NXJ1S0505MC-R13" (at 69.85 160.02 0) (effects (font (size 1.27 1.27))))
+    (property "Footprint" "Converter_DCDC:Converter_DCDC_NXJ1S_SMD" (at 69.85 165.1 0) (effects (font (size 1.27 1.27)) hide))
+    (property "MPN" "NXJ1S0505MC-R13" (at 69.85 165.1 0) (effects (font (size 1.27 1.27)) hide))
+    (property "Manufacturer" "Murata" (at 69.85 165.1 0) (effects (font (size 1.27 1.27)) hide))
+    (property "Description" "1W isolated 5V-5V DC-DC, 5.2kVDC, RS485 bus side" (at 69.85 165.1 0) (effects (font (size 1.27 1.27)) hide))
+  )
+  (symbol (lib_id "Converter_DCDC:NXJ1S0505MC-R13") (at 139.7 165.1) (unit 1)
+    (exclude_from_sim no) (in_bom yes) (on_board yes) (dnp no)
+    (uuid "COM-0015-U43")
+    (property "Reference" "U43" (at 139.7 157.48 0) (effects (font (size 1.27 1.27))))
+    (property "Value" "NXJ1S0505MC-R13" (at 139.7 160.02 0) (effects (font (size 1.27 1.27))))
+    (property "Footprint" "Converter_DCDC:Converter_DCDC_NXJ1S_SMD" (at 139.7 165.1 0) (effects (font (size 1.27 1.27)) hide))
+    (property "MPN" "NXJ1S0505MC-R13" (at 139.7 165.1 0) (effects (font (size 1.27 1.27)) hide))
+    (property "Manufacturer" "Murata" (at 139.7 165.1 0) (effects (font (size 1.27 1.27)) hide))
+    (property "Description" "1W isolated 5V-5V DC-DC, 5.2kVDC, CAN bus side" (at 139.7 165.1 0) (effects (font (size 1.27 1.27)) hide))
+  )
+  (symbol (lib_id "Device:C") (at 62.23 165.1) (unit 1)
+    (exclude_from_sim no) (in_bom yes) (on_board yes) (dnp no)
+    (uuid "COM-0016-C71")
+    (property "Reference" "C71" (at 62.23 163.83 0) (effects (font (size 1.27 1.27))))
+    (property "Value" "10uF" (at 62.23 167.64 0) (effects (font (size 1.27 1.27))))
+    (property "Footprint" "Capacitor_SMD:C_0805_2012Metric" (at 62.23 165.1 0) (effects (font (size 1.27 1.27)) hide))
+    (property "MPN" "GRM21BR61E106KA73L" (at 62.23 165.1 0) (effects (font (size 1.27 1.27)) hide))
+    (property "Manufacturer" "Murata" (at 62.23 165.1 0) (effects (font (size 1.27 1.27)) hide))
+    (property "Description" "+5V input bulk, U42" (at 62.23 165.1 0) (effects (font (size 1.27 1.27)) hide))
+  )
+  (symbol (lib_id "Device:C") (at 78.74 165.1) (unit 1)
+    (exclude_from_sim no) (in_bom yes) (on_board yes) (dnp no)
+    (uuid "COM-0017-C72")
+    (property "Reference" "C72" (at 78.74 163.83 0) (effects (font (size 1.27 1.27))))
+    (property "Value" "10uF" (at 78.74 167.64 0) (effects (font (size 1.27 1.27))))
+    (property "Footprint" "Capacitor_SMD:C_0805_2012Metric" (at 78.74 165.1 0) (effects (font (size 1.27 1.27)) hide))
+    (property "MPN" "GRM21BR61E106KA73L" (at 78.74 165.1 0) (effects (font (size 1.27 1.27)) hide))
+    (property "Manufacturer" "Murata" (at 78.74 165.1 0) (effects (font (size 1.27 1.27)) hide))
+    (property "Description" "RS485_ISO_VCC output bulk" (at 78.74 165.1 0) (effects (font (size 1.27 1.27)) hide))
+  )
+  (symbol (lib_id "Device:C") (at 132.08 165.1) (unit 1)
+    (exclude_from_sim no) (in_bom yes) (on_board yes) (dnp no)
+    (uuid "COM-0018-C73")
+    (property "Reference" "C73" (at 132.08 163.83 0) (effects (font (size 1.27 1.27))))
+    (property "Value" "10uF" (at 132.08 167.64 0) (effects (font (size 1.27 1.27))))
+    (property "Footprint" "Capacitor_SMD:C_0805_2012Metric" (at 132.08 165.1 0) (effects (font (size 1.27 1.27)) hide))
+    (property "MPN" "GRM21BR61E106KA73L" (at 132.08 165.1 0) (effects (font (size 1.27 1.27)) hide))
+    (property "Manufacturer" "Murata" (at 132.08 165.1 0) (effects (font (size 1.27 1.27)) hide))
+    (property "Description" "+5V input bulk, U43" (at 132.08 165.1 0) (effects (font (size 1.27 1.27)) hide))
+  )
+  (symbol (lib_id "Device:C") (at 148.59 165.1) (unit 1)
+    (exclude_from_sim no) (in_bom yes) (on_board yes) (dnp no)
+    (uuid "COM-0019-C74")
+    (property "Reference" "C74" (at 148.59 163.83 0) (effects (font (size 1.27 1.27))))
+    (property "Value" "10uF" (at 148.59 167.64 0) (effects (font (size 1.27 1.27))))
+    (property "Footprint" "Capacitor_SMD:C_0805_2012Metric" (at 148.59 165.1 0) (effects (font (size 1.27 1.27)) hide))
+    (property "MPN" "GRM21BR61E106KA73L" (at 148.59 165.1 0) (effects (font (size 1.27 1.27)) hide))
+    (property "Manufacturer" "Murata" (at 148.59 165.1 0) (effects (font (size 1.27 1.27)) hide))
+    (property "Description" "CAN_ISO_VCC output bulk" (at 148.59 165.1 0) (effects (font (size 1.27 1.27)) hide))
   )
   ;; ============================================================
