File: hardware/kicad/STM32H743_DataLogger/STM32H743_DataLogger.kicad_sch (KiCad schematic)
At the start: 0 parts

Commit message: feat: Add P9E silkscreen branding, fix BOM/schematic cross-check issues
- Add complete silkscreen: P9E branding (3.5mm bold), company name,
  website, product info (Weather Station v2.0), functional area labels,
  connector pin labels, LED labels, compliance marks on back
- Fix BOM: add missing J12/J13/J14/R14-R16, resolve LED4 duplicate
  (renamed to LED5 for BLE), fix C101 conflict with C104
- Complete analog input schematic channels 1-3 (TVS, precision resistors,
  anti-alias RC filter, OPA2376 U21 for Ch2-3)
- Complete digital I/O schematic: add optocouplers U32-U37, current
  limiting resistors, pull-ups R38-R44 for DI Ch1-7, relays K2-K4
- Rebrand all files from SCADA Systems to P9E Microsystems Pvt Ltd
- Update revision to 2.0, date to 2026-03-20

https://claude.ai/code/session_01XsiZ6LJT6X46LKY8yEbRbx
Other:
- company: SCADA Systems -> P9E Microsystems Pvt Ltd
- title: STM32H743 PLC-Grade Data Logger - Top Level -> Weather Station v2.0 - STM32H743 Data Logger
Changed lines of the file:
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@@
   (paper "A3")
   (title_block
-    (title "STM32H743 PLC-Grade Data Logger - Top Level")
-    (date "2026-03-15")
-    (rev "1.0")
-    (company "SCADA Systems")
+    (title "Weather Station v2.0 - STM32H743 Data Logger")
+    (date "2026-03-20")
+    (rev "2.0")
+    (company "P9E Microsystems Pvt Ltd")
     (comment 1 "PLC-Grade Industrial Data Logger")
     (comment 2 "LoRa / BLE / WiFi / Ethernet / GSM")
     (comment 3 "24V Industrial Power Input")
-    (comment 4 "STM32H743VIT6 ARM Cortex-M7 480MHz")
+    (comment 4 "STM32H743VIT6 ARM Cortex-M7 480MHz | www.p9e.in")
   )
   ;; ============================================================
