File: hardware/kicad/STM32H743_DataLogger/Storage.kicad_sch (KiCad schematic)
At the start: 10 parts, among them J80 microSD Slot, U70 W25Q64JVSSIQ, U71 AT24C256C-SSHL-T

Commit message: Complete mfg PCB placement, fix designator conflicts, sync BOM
Manufacturing PCB (STM32H743_DataLogger_mfg.kicad_pcb):
- Add all missing multi-channel footprints: analog channels 1-3
  (D11-D13, R24-R35, C61-C63) plus second op-amp U21
- Add full 8-channel digital input chain (R100-R107 limiters,
  U30/U32-U38 optocouplers, R108-R115 pull-ups) with new
  DI_n_LED nets instead of floating net 0
- Add relays K2-K4 and replace the oversized SANYOU SRD placeholder
  with an HF46F-G/5-HS1T form-A footprint; wire relay contacts to
  J40-J43 via new DOn_NO / DOn_COM nets
- Add C104 (EEPROM decoupling), LED4 + R17 (comm activity indicator)
- Rename the BLE indicator from LED4 to LED5 to match the schematic
- Replace silkscreen branding with the full P9E block (company mark,
  P9E Microsystems Pvt Ltd, www.p9e.in, product, specs) on F.SilkS and
  P/N, S/N, compliance marks and origin on B.SilkS; www.p9e.io and the
  stale "SCADA Systems" text are gone
- Resolve all 26 footprint overlaps, pull the USB-C receptacle fully
  on-board, move fiducials clear of mounting holes, and drop the 22
  stitching vias that landed on pads

Schematics:
- Renumber Digital_IO resistors to R100-R115 and the eighth
  optocoupler to U38, removing the R31x/R40x placeholder designators
  and the R30/R31/R40/R41 collisions with Analog_Inputs and RS485_CAN
- Add C104 to Storage and LED4 + R17 to the MCU sheet

BOM: update the digital I/O and analog designator ranges to match,
add R17, correct the relay type to SPST-NO, and refresh the totals
(116 line items, 211 components).

Co-Authored-By: Claude Opus 5 <noreply@anthropic.com>
Claude-Session: https://claude.ai/code/session_01XsiZ6LJT6X46LKY8yEbRbx
Parts:
- added C104: 100nF, Capacitor_SMD:C_0402_1005Metric, symbol Device:C
Changed lines of the file:
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@@
     (property "Manufacturer" "Murata" (at 69.85 146.05 0) (effects (font (size 1.27 1.27)) hide))
+  )
+  ;; C104 - AT24C256 EEPROM decoupling
+  (symbol (lib_id "Device:C") (at 78.74 146.05) (unit 1)
+    (exclude_from_sim no) (in_bom yes) (on_board yes) (dnp no)
+    (uuid "ST-0021-C104")
+    (property "Reference" "C104" (at 81.28 144.78 0) (effects (font (size 1.27 1.27))))
+    (property "Value" "100nF" (at 78.74 148.59 0) (effects (font (size 1.27 1.27))))
+    (property "Footprint" "Capacitor_SMD:C_0402_1005Metric" (at 78.74 146.05 0) (effects (font (size 1.27 1.27)) hide))
+    (property "MPN" "GRM155R71C104KA88D" (at 78.74 146.05 0) (effects (font (size 1.27 1.27)) hide))
+    (property "Manufacturer" "Murata" (at 78.74 146.05 0) (effects (font (size 1.27 1.27)) hide))
   )
   ;; I2C pull-ups

Commit message: Verify every IC against its datasheet pinout; rebuild three, add missing parts
The MCU turned out not to be the only placeholder. With the symbol
libraries available I checked each IC's footprint wiring against the pin
names its datasheet-derived KiCad symbol gives — if a pin the datasheet
calls VDD is not on a supply net, the map was not derived from the
datasheet. Three ICs failed and are rebuilt:

- U50 W5500 had SPI on the Ethernet differential pins and supplies and
  grounds on ten wrong pads. Rebuilt from the 48-pin pinout: SPI on
  32-37, TX/RX pairs on 1/2/5/6, PMODE2..0 grounded for all-capable
  auto-negotiation.
- U40 ISO3082 had the receiver and driver swapped, the bus A/B pair one
  pin out, and GND2 carrying the isolated 5V supply.
- U1 TPS54560 had the switch node on pins 7 and 8, shorting SW to GND,
  and FB off pin 5.

Verifying the W5500 also showed three datasheet-required parts were never
placed: R56 (12.4k on EXRES1, sets transmit bias current), C87 (4.7uF on
TOCAP) and C88 (100nF on VBG). All three added.

Two ICs cannot be verified and are recorded as such rather than guessed
at. U60 is worse than a wiring error: the footprint is QFN-28 4x4mm on
0.4mm pitch, but SX1276IMLTRT is 6x6mm on 0.65mm pitch — the wrong
package outline entirely. U3's part is the DGN (MSOP-8-EP) variant and
the library only has KTT (TO-263-5), a different pinout, so it cannot
stand in. Six more ICs have no symbol at all and show the same sequential
pattern; they should be assumed wrong until checked.

Still open on the buck: EN, RT/CLK and COMP have no components on them.
RT/CLK sets the switching frequency and COMP is the compensation network,
so U1 will not regulate as drawn.

Also corrected twelve wrong schematic lib_ids against the real libraries;
35 of 44 now resolve, and the nine that need symbols drawn are listed in
docs/Schematic_Symbol_Audit.md.

BOM now 123 line items / 222 components; netlist 160 nets, all reaching
at least two pads.

Co-Authored-By: Claude O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
Parts:
- J80: symbol Connector:Micro_SD_Card_Det -> Connector:Micro_SD_Card_Det1
- U71: symbol Memory_EEPROM:AT24C256C -> Memory_EEPROM:CAT24C256
Changed lines of the file:
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@@
   ;; ============================================================
   (symbol
-    (lib_id "Connector:Micro_SD_Card_Det")
+    (lib_id "Connector:Micro_SD_Card_Det1")
     (at 88.9 57.15)
     (unit 1)
@@
   ;; ============================================================
   (symbol
-    (lib_id "Memory_EEPROM:AT24C256C")
+    (lib_id "Memory_EEPROM:CAT24C256")
     (at 88.9 152.4)
     (unit 1)
