File: hardware/kicad/STM32H743_DataLogger/Wireless.kicad_sch (KiCad schematic)
At the start: 18 parts, among them J70 SMA LoRa ANT, J71 U.FL WiFi/BLE ANT, J72 Nano SIM Holder, J73 SMA LTE Main ANT, J74 SMA GNSS ANT, U60 RFM95W-915S2, U61 ESP32-C3-MINI-1-N4, U62 SIM7600G-H, U63 TPS73641DCQR

Commit message: feat: Upgrade to full industrial-grade components and SPI architecture
Major design changes for PLC-grade reliability:

Component Upgrades:
- Replace ESP32-C3 dual-MCU with ATWINC1500 WiFi (SPI2) + RN4870 BLE (UART7)
  Eliminates second processor, both rated -40 to +85°C industrial
- Replace LAN8742A RMII PHY with W5500 SPI Ethernet controller
  Hardwired TCP/IP stack, frees 11 RMII pins, simpler firmware
- Replace RFM95W module with SX1276IMLTRT bare IC (-40 to +85°C)
  Full industrial temp range with 32MHz TCXO and custom RF matching
- Add TPS3823-33 external hardware watchdog (1.6s timeout)

Industrial Compliance:
- All key ICs rated -40 to +85°C (industrial grade)
- HumiSeal 1B73 conformal coating spec (MIL-I-46058C)
- EMC compliance targets: IEC 61000-4-2/4/5/6/8
- Ferrite beads on Ethernet pairs for EMI

Architecture: Single MCU (STM32H743) with all peripherals as SPI/UART slaves
- SPI1: SX1276 LoRa
- SPI2: ATWINC1500 WiFi
- SPI3: W25Q64JV Flash
- SPI4: W5500 Ethernet
- UART4: SIM7600G-H GSM/LTE
- UART7: RN4870 BLE

Updated BOM: ~170 components, ~$142/unit (1pc), ~$90/unit (100pc)

https://claude.ai/code/session_01XsiZ6LJT6X46LKY8yEbRbx
Parts:
- added C90B: 5.6pF C0G, Capacitor_SMD:C_0402_1005Metric, symbol Device:C
- added C90C: 6.8pF C0G, Capacitor_SMD:C_0402_1005Metric, symbol Device:C
- added C93B, C94A, C97, C98: 100nF, Capacitor_SMD:C_0402_1005Metric, symbol Device:C
- added C96: 10uF, Capacitor_SMD:C_0805_2012Metric, symbol Device:C
- added LED4: Blue BLE, LED_SMD:LED_0603_1608Metric, symbol Device:LED
- added R61, R62, R63, R64: 10k, Resistor_SMD:R_0402_1005Metric, symbol Device:R
- added R65: 1k, Resistor_SMD:R_0402_1005Metric, symbol Device:R
- added U62B: RN4870-I/RM128, RF_Bluetooth:Microchip_RN4870, symbol RF_Bluetooth:RN4870
- added U64: TPS3823-33DBVR, Package_TO_SOT_SMD:SOT-23-5, symbol Timer:TPS3823
- added Y4: 32MHz TCXO, Crystal:Crystal_SMD_2016-4Pin_2.0x1.6mm, symbol Device:Crystal
- J71: value U.FL WiFi/BLE ANT -> U.FL WiFi ANT
- U60: value RFM95W-915S2 -> SX1276IMLTRT; footprint RF_Module:HOPERF_RFM9XW_SMD -> Package_DFN_QFN:QFN-28-1EP_4x4mm_P0.4mm_EP2.4x2.4mm; MPN RFM95W-915S2 -> SX1276IMLTRT; Manufacturer HopeRF -> Semtech
- U61: value ESP32-C3-MINI-1-N4 -> ATWINC1500-MR210PB1952; footprint RF_Module:ESP32-C3-MINI-1 -> RF_Module:Microchip_ATWINC15x0-MR210xB; symbol RF_Module:ESP32-C3-MINI-1 -> RF_WiFi:ATWINC1500-MR210PB; MPN ESP32-C3-MINI-1-N4 -> ATWINC1500-MR210PB1952; Manufacturer Espressif -> Microchip
Other:
- note added: "WIRELESS COMMUNICATIONS (Rev 1.2 - Full Industrial Grade) 1. LoRa (SX1276IMLTRT - Bare IC): - SPI1 interface, 868/915MHz - +20dBm TX, -148dBm sensitivity - SMA antenna connector + pi-matching network - INDUSTRIAL TEMP: -40 to +85C (bare IC, not module) - QFN-28 package, custom RF section with matching - 32MHz TCXO for frequency stability 2. WiFi (ATWINC1500-MR210PB): - SPI2 interface, 802.11 b/g/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"
- note removed: "WIRELESS COMMUNICATIONS 1. LoRa (SX1276/RFM95W): - SPI1 interface, 868/915MHz - +20dBm TX, -148dBm sensitivity - SMA antenna connector - Range: up to 15km LOS 2. BLE + WiFi (ESP32-C3-MINI-1): - WiFi 802.11 b/g/n (2.4GHz) - Bluetooth 5.0 LE - UART7 for AT commands - u.FL antenna connector 3. GSM/LTE (SIM7600G-H): - LTE Cat-1 global bands - 2G/3G fallback - UART4 interface, AT commands - Nano SIM p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"
- title: Wireless Communications - LoRa, BLE, WiFi, GSM -> Wireless Communications - LoRa, WiFi, BLE, GSM

Commit message: feat: Add P9E silkscreen branding, fix BOM/schematic cross-check issues
- Add complete silkscreen: P9E branding (3.5mm bold), company name,
  website, product info (Weather Station v2.0), functional area labels,
  connector pin labels, LED labels, compliance marks on back
- Fix BOM: add missing J12/J13/J14/R14-R16, resolve LED4 duplicate
  (renamed to LED5 for BLE), fix C101 conflict with C104
- Complete analog input schematic channels 1-3 (TVS, precision resistors,
  anti-alias RC filter, OPA2376 U21 for Ch2-3)
- Complete digital I/O schematic: add optocouplers U32-U37, current
  limiting resistors, pull-ups R38-R44 for DI Ch1-7, relays K2-K4
- Rebrand all files from SCADA Systems to P9E Microsystems Pvt Ltd
- Update revision to 2.0, date to 2026-03-20

https://claude.ai/code/session_01XsiZ6LJT6X46LKY8yEbRbx
Parts:
- removed LED4: Blue BLE, LED_SMD:LED_0603_1608Metric, symbol Device:LED
- added LED5: Blue BLE, LED_SMD:LED_0603_1608Metric, symbol Device:LED
Other:
- company: SCADA Systems -> P9E Microsystems Pvt Ltd
Changed lines of the file:
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@@
     (date "2026-03-15")
     (rev "1.1")
-    (company "SCADA Systems")
+    (company "P9E Microsystems Pvt Ltd")
     (comment 1 "LoRa: RFM95W (SPI1) | WiFi: ATWINC1500 (SPI2) | BLE: RN4870 (UART7)")
     (comment 2 "GSM/LTE: SIM7600G-H (UART4) with SIM card holder")
@@
   (symbol (lib_id "Device:LED") (at 215.9 57.15) (unit 1)
     (exclude_from_sim no) (in_bom yes) (on_board yes) (dnp no)
-    (uuid "WL-0034-LED4")
-    (property "Reference" "LED4" (at 215.9 52.07 0) (effects (font (size 1.27 1.27))))
+    (uuid "WL-0034-LED5")
+    (property "Reference" "LED5" (at 215.9 52.07 0) (effects (font (size 1.27 1.27))))
     (property "Value" "Blue BLE" (at 215.9 54.61 0) (effects (font (size 1.27 1.27))))
     (property "Footprint" "LED_SMD:LED_0603_1608Metric" (at 215.9 57.15 0) (effects (font (size 1.27 1.27)) hide))
