File: hardware/kicad/STM32H743_DataLogger/Wireless.kicad_sch (KiCad schematic)
At the start: 34 parts, among them J70 SMA LoRa ANT, J71 U.FL WiFi ANT, J72 Nano SIM Holder, J73 SMA LTE Main ANT, J74 SMA GNSS ANT, U60 SX1276IMLTRT, U61 ATWINC1500-MR210PB1952, U62 SIM7600G-H, U62B RN4870-I/RM128, U63 TPS73641DCQR, U64 TPS3823-33DBVR, Y4 32MHz TCXO

Commit message: Close six unconnected nets found while exporting the netlist
Exporting the board to Specctra for routing surfaced six nets with only
one pad on them — they had nothing to connect to:

- VBUCK_BST reached only U1 pin 1. The buck had no bootstrap capacitor,
  so the high-side switch could never turn on and the 24V-to-5V stage
  would not start. Added C11 (100nF) from BST to the SW node.
- USART1_TX_BUF and USART1_RX_BUF dead-ended at R14/R15. J12 tapped the
  MCU side of the 33R series resistors, so the debug header was wired
  straight to the MCU and the resistors sat in mid-air. J12 now taps the
  buffered side, putting them in circuit as intended.
- GSM_DTR, GSM_RI and LORA_DIO1 reached only their module pins. The MCU
  has no spare pad (all 100 are assigned), so DTR gets a 10k pull-down
  (R18) to hold the modem out of sleep rather than floating, and RI and
  DIO1 come out to probe pads TP9/TP10.

Also added TP1-TP8 to the schematics; they existed only as PCB pads, so
the netlist and the board disagreed about them.

BOM now 120 line items / 219 components. Placement re-verified: 227
footprints, zero courtyard collisions, nothing off-board.

Co-Authored-By: Claude Opus 5 <noreply@anthropic.com>
Claude-Session: https://claude.ai/code/session_01XsiZ6LJT6X46LKY8yEbRbx
Parts:
- added R18: 10k, Resistor_SMD:R_0402_1005Metric, symbol Device:R
- added TP10: LORA_DIO1, TestPoint:TestPoint_Pad_1.0x1.0mm, symbol Connector:TestPoint
- added TP9: GSM_RI, TestPoint:TestPoint_Pad_1.0x1.0mm, symbol Connector:TestPoint
Changed lines of the file:
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@@
     (uuid "WL-TEXT-0001")
   )
+  ;; R18 - SIM7600 DTR pull-down: no spare MCU pin, so hold the modem awake.
+  (symbol (lib_id "Device:R") (at 190.5 165.1) (unit 1)
+    (exclude_from_sim no) (in_bom yes) (on_board yes) (dnp no)
+    (uuid "WL-0050-R18")
+    (property "Reference" "R18" (at 193.04 165.1 0) (effects (font (size 1.27 1.27))))
+    (property "Value" "10k" (at 190.5 167.64 0) (effects (font (size 1.27 1.27))))
+    (property "Footprint" "Resistor_SMD:R_0402_1005Metric" (at 190.5 165.1 0) (effects (font (size 1.27 1.27)) hide))
+    (property "MPN" "RC0402FR-0710KL" (at 190.5 165.1 0) (effects (font (size 1.27 1.27)) hide))
+    (property "Manufacturer" "Yageo" (at 190.5 165.1 0) (effects (font (size 1.27 1.27)) hide))
+  )
+  (symbol (lib_id "Connector:TestPoint") (at 203.2 165.1) (unit 1)
+    (exclude_from_sim no) (in_bom yes) (on_board yes) (dnp no)
+    (uuid "WL-0051-TP9")
+    (property "Reference" "TP9" (at 203.2 161.29 0) (effects (font (size 1.27 1.27))))
+    (property "Value" "GSM_RI" (at 203.2 163.83 0) (effects (font (size 1.27 1.27))))
+    (property "Footprint" "TestPoint:TestPoint_Pad_1.0x1.0mm" (at 203.2 165.1 0) (effects (font (size 1.27 1.27)) hide))
+  )
+  (symbol (lib_id "Connector:TestPoint") (at 215.9 165.1) (unit 1)
+    (exclude_from_sim no) (in_bom yes) (on_board yes) (dnp no)
+    (uuid "WL-0052-TP10")
+    (property "Reference" "TP10" (at 215.9 161.29 0) (effects (font (size 1.27 1.27))))
+    (property "Value" "LORA_DIO1" (at 215.9 163.83 0) (effects (font (size 1.27 1.27))))
+    (property "Footprint" "TestPoint:TestPoint_Pad_1.0x1.0mm" (at 215.9 165.1 0) (effects (font (size 1.27 1.27)) hide))
+  )
 )

Commit message: Verify every IC against its datasheet pinout; rebuild three, add missing parts
The MCU turned out not to be the only placeholder. With the symbol
libraries available I checked each IC's footprint wiring against the pin
names its datasheet-derived KiCad symbol gives — if a pin the datasheet
calls VDD is not on a supply net, the map was not derived from the
datasheet. Three ICs failed and are rebuilt:

- U50 W5500 had SPI on the Ethernet differential pins and supplies and
  grounds on ten wrong pads. Rebuilt from the 48-pin pinout: SPI on
  32-37, TX/RX pairs on 1/2/5/6, PMODE2..0 grounded for all-capable
  auto-negotiation.
- U40 ISO3082 had the receiver and driver swapped, the bus A/B pair one
  pin out, and GND2 carrying the isolated 5V supply.
- U1 TPS54560 had the switch node on pins 7 and 8, shorting SW to GND,
  and FB off pin 5.

Verifying the W5500 also showed three datasheet-required parts were never
placed: R56 (12.4k on EXRES1, sets transmit bias current), C87 (4.7uF on
TOCAP) and C88 (100nF on VBG). All three added.

Two ICs cannot be verified and are recorded as such rather than guessed
at. U60 is worse than a wiring error: the footprint is QFN-28 4x4mm on
0.4mm pitch, but SX1276IMLTRT is 6x6mm on 0.65mm pitch — the wrong
package outline entirely. U3's part is the DGN (MSOP-8-EP) variant and
the library only has KTT (TO-263-5), a different pinout, so it cannot
stand in. Six more ICs have no symbol at all and show the same sequential
pattern; they should be assumed wrong until checked.

Still open on the buck: EN, RT/CLK and COMP have no components on them.
RT/CLK sets the switching frequency and COMP is the compensation network,
so U1 will not regulate as drawn.

Also corrected twelve wrong schematic lib_ids against the real libraries;
35 of 44 now resolve, and the nine that need symbols drawn are listed in
docs/Schematic_Symbol_Audit.md.

BOM now 123 line items / 222 components; netlist 160 nets, all reaching
at least two pads.

Co-Authored-By: Claude O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
Parts:
- U60: symbol RF_Module:RFM95W-868S2 -> RF_Module:SX1276
- U64: symbol Timer:TPS3823 -> Power_Supervisor:TPS3823-xxDBV
Changed lines of the file:
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@@
   ;; ============================================================
   (symbol
-    (lib_id "RF_Module:RFM95W-868S2")
+    (lib_id "RF_Module:SX1276")
     (at 76.2 63.5)
     (unit 1)
@@
   ;; ============================================================
   (symbol
-    (lib_id "Timer:TPS3823")
+    (lib_id "Power_Supervisor:TPS3823-xxDBV")
     (at 190.5 133.35)
     (unit 1)
