File: hardware/kicad/STM32H743_DataLogger/STM32H743_DataLogger_mfg.kicad_pcb (KiCad board)
At the start: 4 copper layers, 160 x 100 mm, 224 parts, among them J1 24VDC_Input, J10 SWD_Debug, J11 USB-C, J12 UART_Debug, J13 BOOT0_Select, J14 TC2050-IDC, J20 AI_CH0, J21 AI_CH1, J22 AI_CH2, J23 AI_CH3, J30 DI_0, J31 DI_1, J32 DI_2, J33 DI_3, J34 DI_4, J35 DI_5, J36 DI_6, J37 DI_7, J40 DO_0, J41 DO_1, J42 DO_2, J43 DO_3, J50 RS485, J51 CAN, J60 J0011D21BNL, J70 SMA_LoRa, J71 U.FL_WiFi, J72 NanoSIM, J73 SMA_LTE, J74 SMA_GNSS, J80 microSD, K1 HF46F-G/5-HS1T, K2 HF46F-G/5-HS1T, K3 HF46F-G/5-HS1T, K4 HF46F-G/5-HS1T, Q1 SI4435DDY, U1 TPS54560, U10 STM32H743VIT6, U2 TLV1117LV33, U20 OPA2376, U21 OPA2376, U3 TPS7A4533, U30 TLP293, U31 ULN2003A, U32 TLP293, U33 TLP293, U34 TLP293, U35 TLP293, U36 TLP293, U37 TLP293, U38 TLP293, U40 ISO3082, U41 ISO1042, U42 NXJ1S0505MC, U43 NXJ1S0505MC, U50 W5500, U60 SX1276, U61 ATWINC1500, U62 SIM7600G-H, U62B RN4870, U63 TPS73641, U64 TPS3823-33, U70 W25Q64JV, U71 AT24C256C, Y1 25MHz, Y2 32.768kHz, Y3 25MHz, Y4 32MHz

Commit message: Close six unconnected nets found while exporting the netlist
Exporting the board to Specctra for routing surfaced six nets with only
one pad on them — they had nothing to connect to:

- VBUCK_BST reached only U1 pin 1. The buck had no bootstrap capacitor,
  so the high-side switch could never turn on and the 24V-to-5V stage
  would not start. Added C11 (100nF) from BST to the SW node.
- USART1_TX_BUF and USART1_RX_BUF dead-ended at R14/R15. J12 tapped the
  MCU side of the 33R series resistors, so the debug header was wired
  straight to the MCU and the resistors sat in mid-air. J12 now taps the
  buffered side, putting them in circuit as intended.
- GSM_DTR, GSM_RI and LORA_DIO1 reached only their module pins. The MCU
  has no spare pad (all 100 are assigned), so DTR gets a 10k pull-down
  (R18) to hold the modem out of sleep rather than floating, and RI and
  DIO1 come out to probe pads TP9/TP10.

Also added TP1-TP8 to the schematics; they existed only as PCB pads, so
the netlist and the board disagreed about them.

BOM now 120 line items / 219 components. Placement re-verified: 227
footprints, zero courtyard collisions, nothing off-board.

Co-Authored-By: Claude Opus 5 <noreply@anthropic.com>
Claude-Session: https://claude.ai/code/session_01XsiZ6LJT6X46LKY8yEbRbx
Parts:
- added C11: 100nF, Capacitor_SMD:C_0402_1005Metric, F.Cu at (38.5, 46.0)
- added R18: 10k, Resistor_SMD:R_0402_1005Metric, F.Cu at (116.0, 30.5)
- added TP10: LORA_DIO1, TestPoint:TestPoint_Pad_1.0x1.0mm, F.Cu at (129.0, 69.5)
- added TP9: GSM_RI, TestPoint:TestPoint_Pad_1.0x1.0mm, F.Cu at (99.5, 47.0)
Connections:
- J12 pad 2: USART1_TX -> USART1_TX_BUF
- J12 pad 3: USART1_RX -> USART1_RX_BUF
Changed lines of the file:
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@@
     (property "Value" "UART_Debug" (at 0 3) (layer "F.Fab") (effects (font (size 0.8 0.8) (thickness 0.12))))
     (pad "1" thru_hole rect (at 0 0) (size 1.7 1.7) (drill 1) (layers "*.Cu" "*.Mask") (net 2 "+3V3"))
-    (pad "2" thru_hole circle (at 0 2.54) (size 1.7 1.7) (drill 1) (layers "*.Cu" "*.Mask") (net 35 "USART1_TX"))
-    (pad "3" thru_hole circle (at 0 5.08) (size 1.7 1.7) (drill 1) (layers "*.Cu" "*.Mask") (net 36 "USART1_RX"))
+    (pad "2" thru_hole circle (at 0 2.54) (size 1.7 1.7) (drill 1) (layers "*.Cu" "*.Mask") (net 103 "USART1_TX_BUF"))
+    (pad "3" thru_hole circle (at 0 5.08) (size 1.7 1.7) (drill 1) (layers "*.Cu" "*.Mask") (net 104 "USART1_RX_BUF"))
     (pad "4" thru_hole circle (at 0 7.62) (size 1.7 1.7) (drill 1) (layers "*.Cu" "*.Mask") (net 1 "GND"))
     (fp_rect (start -1.100 -1.100) (end 1.100 8.720) (stroke (width 0.05) (type solid)) (fill none) (layer "F.CrtYd") (uuid "MFG-MCU-J12-CY"))
@@
   )
   ;; ============================================================
+  ;; DANGLING-NET FIXES
+  ;; ============================================================
+  (footprint "Capacitor_SMD:C_0402_1005Metric" (layer "F.Cu") (uuid "MFG-PS-C11") (at 38.5 46)
+    (property "Reference" "C11" (at 0 -1.2) (layer "F.SilkS") (effects (font (size 0.5 0.5) (thickness 0.08))))
+    (property "Value" "100nF" (at 0 1.2) (layer "F.Fab") (effects (font (size 0.5 0.5) (thickness 0.08))))
+    (pad "1" smd roundrect (at -0.51 0) (size 0.54 0.64) (layers "F.Cu" "F.Paste" "F.Mask") (roundrect_rratio 0.25) (net 92 "VBUCK_BST"))
+    (pad "2" smd roundrect (at 0.51 0) (size 0.54 0.64) (layers "F.Cu" "F.Paste" "F.Mask") (roundrect_rratio 0.25) (net 91 "VBUCK_SW"))
+    (fp_rect (start -1 -0.55) (end 1 0.55) (stroke (width 0.05) (type solid)) (fill none) (layer "F.CrtYd") (uuid "MFG-PS-C11-CY"))
+  )
+  (footprint "Resistor_SMD:R_0402_1005Metric" (layer "F.Cu") (uuid "MFG-WL-R18") (at 116 30.5)
+    (property "Reference" "R18" (at 0 -1.2) (layer "F.SilkS") (effects (font (size 0.5 0.5) (thickness 0.08))))
+    (property "Value" "10k" (at 0 1.2) (layer "F.Fab") (effects (font (size 0.5 0.5) (thickness 0.08))))
+    (pad "1" smd roundrect (at -0.51 0) (size 0.54 0.64) (layers "F.Cu" "F.Paste" "F.Mask") (roundrect_rratio 0.25) (net 142 "GSM_DTR"))
+    (pad "2" smd roundrect (at 0.51 0) (size 0.54 0.64) (layers "F.Cu" "F.Paste" "F.Mask") (roundrect_rratio 0.25) (net 1 "GND"))
+    (fp_rect (start -1 -0.55) (end 1 0.55) (stroke (width 0.05) (type solid)) (fill none) (layer "F.CrtYd") (uuid "MFG-WL-R18-CY"))
+  )
+  (footprint "TestPoint:TestPoint_Pad_1.0x1.0mm" (layer "F.Cu") (uuid "MFG-WL-TP9") (at 99.5 47)
+    (property "Reference" "TP9" (at 0 -1.4) (layer "F.SilkS") (effects (font (size 0.5 0.5) (thickness 0.08))))
+    (property "Value" "GSM_RI" (at 0 1.4) (layer "F.Fab") (effects (font (size 0.5 0.5) (thickness 0.08))))
+    (pad "1" smd roundrect (at 0 0) (size 1.0 1.0) (layers "F.Cu" "F.Paste" "F.Mask") (roundrect_rratio 0.25) (net 143 "GSM_RI"))
+    (fp_rect (start -0.8 -0.8) (end 0.8 0.8) (stroke (width 0.05) (type solid)) (fill none) (layer "F.CrtYd") (uuid "MFG-WL-TP9-CY"))
+  )
+  (footprint "TestPoint:TestPoint_Pad_1.0x1.0mm" (layer "F.Cu") (uuid "MFG-WL-TP10") (at 129 69.5)
+    (property "Reference" "TP10" (at 0 -1.4) (layer "F.SilkS") (effects (font (size 0.5 0.5) (thickness 0.08))))
+    (property "Value" "LORA_DIO1" (at 0 1.4) (layer "F.Fab") (effects (font (size 0.5 0.5) (thickness 0.08))))
+    (pad "1" smd roundrect (at 0 0) (size 1.0 1.0) (layers "F.Cu" "F.Paste" "F.Mask") (roundrect_rratio 0.25) (net 141 "LORA_DIO1"))
+    (fp_rect (start -0.8 -0.8) (end 0.8 0.8) (stroke (width 0.05) (type solid)) (fill none) (layer "F.CrtYd") (uuid "MFG-WL-TP10-CY"))
+  )
+  ;; ============================================================

Commit message: Fix J1, re-site the probe pads, refresh the docs to match the board
J1, the 24VDC input, was written with its footprint header split across two
lines. Every check I had run parsed footprints with a single-line header,
so J1 was silently skipped by all of them: it never got a courtyard, the
floorplan pass never moved it, and it was invisible to the collision and
off-board checks. It was still sitting at its original (10, 98) — hanging
3.8mm past the bottom edge and overlapping mounting hole H3 — and it was
also missing from the netlist export, so +24V would not have routed to it.
Header normalised, courtyard added, placed at the head of the bottom
terminal row. It was the only footprint written that way; the checker now
sees all 228.

The probe pads had been packed into whatever region they landed in rather
than placed deliberately — BOOT0 ended up in the relay bank and NRST in the
fieldbus corner. TP1-TP4 now sit with the regulators they measure and
TP5-TP8 with the MCU/SWD signals.

Docs regenerated from the board rather than left at their old coordinates:
fiducial and test-point tables, a new isolation section giving the barrier
line, the four milled slot positions, the pour geometry and the clearances
actually achieved (8mm outer, 7mm below, 4mm between domains — flagged for
check against the datasheets), and a floorplan section describing the edge
assignment and why the two mid-edge mounting holes moved.

Verified: 228 footprints, zero courtyard collisions, nothing off-board.

Co-Authored-By: Claude Opus 5 <noreply@anthropic.com>
Claude-Session: https://claude.ai/code/session_01XsiZ6LJT6X46LKY8yEbRbx
Parts:
- moved J1 6.05 mm to (14.5, 94.0)
Changed lines of the file:
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@@
   ;; ============================================================
   ;; J1 - 24VDC Power Input Terminal Block (bottom edge)
-  (footprint "TerminalBlock_Phoenix:TerminalBlock_Phoenix_MKDS-1,5-2-5.08_1x02_P5.08mm_Horizontal"
-    (layer "F.Cu") (uuid "MFG-PS-J1") (at 10 98)
+  (footprint "TerminalBlock_Phoenix:TerminalBlock_Phoenix_MKDS-1,5-2-5.08_1x02_P5.08mm_Horizontal" (layer "F.Cu") (uuid "MFG-PS-J1") (at 14.54 94)
     (property "Reference" "J1" (at 0 -4) (layer "F.SilkS") (effects (font (size 1 1) (thickness 0.15))))
     (property "Value" "24VDC_Input" (at 0 4) (layer "F.Fab") (effects (font (size 1 1) (thickness 0.15))))
     (pad "1" thru_hole circle (at 0 0) (size 2.4 2.4) (drill 1.3) (layers "*.Cu" "*.Mask") (net 4 "+24V"))
     (pad "2" thru_hole circle (at 5.08 0) (size 2.4 2.4) (drill 1.3) (layers "*.Cu" "*.Mask") (net 1 "GND"))
+    (fp_rect (start -2.54 -4) (end 7.62 5.6) (stroke (width 0.05) (type solid)) (fill none) (layer "F.CrtYd") (uuid "MFG-PS-J1-CY"))
   )
   ;; F1 - PTC Fuse 1.5A
