File: hardware/kicad/STM32H743_DataLogger/STM32H743_DataLogger_mfg.kicad_pcb (KiCad board)
At the start: 4 copper layers, 160 x 100 mm, 231 parts, among them J1 24VDC_Input, J10 SWD_Debug, J11 USB-C, J12 UART_Debug, J13 BOOT0_Select, J14 TC2050-IDC, J20 AI_CH0, J21 AI_CH1, J22 AI_CH2, J23 AI_CH3, J30 DI_0, J31 DI_1, J32 DI_2, J33 DI_3, J34 DI_4, J35 DI_5, J36 DI_6, J37 DI_7, J40 DO_0, J41 DO_1, J42 DO_2, J43 DO_3, J50 RS485, J51 CAN, J60 J0011D21BNL, J70 SMA_LoRa, J71 U.FL_WiFi, J72 NanoSIM, J73 SMA_LTE, J74 SMA_GNSS, J80 microSD, K1 HF46F-G/5-HS1T, K2 HF46F-G/5-HS1T, K3 HF46F-G/5-HS1T, K4 HF46F-G/5-HS1T, Q1 SI4435DDY, U1 TPS54560, U10 STM32H743VIT6, U2 TLV1117LV33, U20 OPA2376, U21 OPA2376, U3 TPS7A4533, U30 TLP293, U31 ULN2003A, U32 TLP293, U33 TLP293, U34 TLP293, U35 TLP293, U36 TLP293, U37 TLP293, U38 TLP293, U40 ISO3082, U41 ISO1042, U42 NXJ1S0505MC, U43 NXJ1S0505MC, U50 W5500, U60 SX1276, U61 ATWINC1500, U62 SIM7600G-H, U62B RN4870, U63 TPS73641, U64 TPS3823-33, U70 W25Q64JV, U71 AT24C256C, Y1 25MHz, Y2 32.768kHz, Y3 25MHz, Y4 32MHz

Commit message: Rewire the analog input buffers; they were shorted and mis-supplied
Following symbol inheritance in the audit (several symbols derive from a
parent via `extends`, so their pins were never actually being read)
exposed the OPA2376 buffers on U20 and U21.

Two faults. Supply and output were swapped: pin 8 is V+ but carried an
ADC signal, while pin 7 (OUT_B) held +3V3A — the amplifier had no supply
and an output pin driving into the rail. And each buffer had its input
and output on a single net, shorting it and leaving the amplifier sitting
in parallel with the ADC node rather than in series with it, so the
conditioned signal never passed through a buffer at all.

Rewired as proper unity-gain buffers: the 1k series resistor and its
100nF cap now form the anti-alias filter on a new AI_CHn_IN node feeding
+IN, with OUT tied back to -IN and on to the ADC pin, V+ on +3V3A and V-
on GND.

The same inheritance fix showed U63 (TPS73641, a 4.1V LDO) is sharing the
TLV1117-33 symbol, which is a different part — its IN and GND look
swapped against that symbol, but the symbol is wrong so the reading is
untrustworthy. Recorded rather than acted on. U2 uses the same symbol and
genuinely is a TLV1117; it checks out clean.

Netlist now 164 nets, all reaching at least two pads. Placement
re-verified: 231 footprints, zero collisions, nothing off-board.

Co-Authored-By: Claude Opus 5 <noreply@anthropic.com>
Claude-Session: https://claude.ai/code/session_01XsiZ6LJT6X46LKY8yEbRbx
Connections:
- C60 pad 1: ADC1_CH0 -> AI_CH0_IN
- C61 pad 1: ADC1_CH1 -> AI_CH1_IN
- C62 pad 1: ADC1_CH2 -> AI_CH2_IN
- C63 pad 1: ADC1_CH3 -> AI_CH3_IN
- R23 pad 2: ADC1_CH0 -> AI_CH0_IN
- R27 pad 2: ADC1_CH1 -> AI_CH1_IN
- R31 pad 2: ADC1_CH2 -> AI_CH2_IN
- R35 pad 2: ADC1_CH3 -> AI_CH3_IN
- U20 pad 3: ADC1_CH1 -> AI_CH0_IN
- U20 pad 5: ADC1_CH1 -> AI_CH1_IN
- U20 pad 7: +3V3A -> ADC1_CH1
- U20 pad 8: ADC1_CH0 -> +3V3A
- U21 pad 3: ADC1_CH3 -> AI_CH2_IN
- U21 pad 5: ADC1_CH3 -> AI_CH3_IN
- U21 pad 7: +3V3A -> ADC1_CH3
- U21 pad 8: ADC1_CH2 -> +3V3A
Changed lines of the file:
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@@
   (net 167 "W5500_TOCAP")
   (net 168 "W5500_VBG")
+  (net 169 "AI_CH0_IN")
+  (net 170 "AI_CH1_IN")
+  (net 171 "AI_CH2_IN")
+  (net 172 "AI_CH3_IN")
   ;; ============================================================
   ;; BOARD OUTLINE - 160x100mm with 3mm corner radius
@@
     (property "Value" "1k" (at 0 1.2) (layer "F.Fab") (effects (font (size 0.5 0.5) (thickness 0.08))))
     (pad "1" smd roundrect (at -0.51 0) (size 0.54 0.64) (layers "F.Cu" "F.Paste" "F.Mask") (roundrect_rratio 0.25) (net 118 "AI_CH0_FILT"))
-    (pad "2" smd roundrect (at 0.51 0) (size 0.54 0.64) (layers "F.Cu" "F.Paste" "F.Mask") (roundrect_rratio 0.25) (net 62 "ADC1_CH0"))
+    (pad "2" smd roundrect (at 0.51 0) (size 0.54 0.64) (layers "F.Cu" "F.Paste" "F.Mask") (roundrect_rratio 0.25) (net 169 "AI_CH0_IN"))
     (fp_rect (start -1.030 -0.570) (end 1.030 0.570) (stroke (width 0.05) (type solid)) (fill none) (layer "F.CrtYd") (uuid "MFG-AI-R23-CY"))
   )
@@
     (property "Reference" "C60" (at 0 -1.2) (layer "F.SilkS") (effects (font (size 0.5 0.5) (thickness 0.08))))
     (property "Value" "100nF" (at 0 1.2) (layer "F.Fab") (effects (font (size 0.5 0.5) (thickness 0.08))))
-    (pad "1" smd roundrect (at -0.51 0) (size 0.54 0.64) (layers "F.Cu" "F.Paste" "F.Mask") (roundrect_rratio 0.25) (net 62 "ADC1_CH0"))
+    (pad "1" smd roundrect (at -0.51 0) (size 0.54 0.64) (layers "F.Cu" "F.Paste" "F.Mask") (roundrect_rratio 0.25) (net 169 "AI_CH0_IN"))
     (pad "2" smd roundrect (at 0.51 0) (size 0.54 0.64) (layers "F.Cu" "F.Paste" "F.Mask") (roundrect_rratio 0.25) (net 1 "GND"))
     (fp_rect (start -1.030 -0.570) (end 1.030 0.570) (stroke (width 0.05) (type solid)) (fill none) (layer "F.CrtYd") (uuid "MFG-AI-C60-CY"))
@@
     (pad "1" smd roundrect (at -2.1 -0.975) (size 1.4 0.45) (layers "F.Cu" "F.Paste" "F.Mask") (roundrect_rratio 0.25) (net 62 "ADC1_CH0"))
     (pad "2" smd roundrect (at -2.1 -0.325) (size 1.4 0.45) (layers "F.Cu" "F.Paste" "F.Mask") (roundrect_rratio 0.25) (net 62 "ADC1_CH0"))
-    (pad "3" smd roundrect (at -2.1 0.325) (size 1.4 0.45) (layers "F.Cu" "F.Paste" "F.Mask") (roundrect_rratio 0.25) (net 63 "ADC1_CH1"))
+    (pad "3" smd roundrect (at -2.1 0.325) (size 1.4 0.45) (layers "F.Cu" "F.Paste" "F.Mask") (roundrect_rratio 0.25) (net 169 "AI_CH0_IN"))
     (pad "4" smd roundrect (at -2.1 0.975) (size 1.4 0.45) (layers "F.Cu" "F.Paste" "F.Mask") (roundrect_rratio 0.25) (net 1 "GND"))
-    (pad "5" smd roundrect (at 2.1 0.975) (size 1.4 0.45) (layers "F.Cu" "F.Paste" "F.Mask") (roundrect_rratio 0.25) (net 63 "ADC1_CH1"))
+    (pad "5" smd roundrect (at 2.1 0.975) (size 1.4 0.45) (layers "F.Cu" "F.Paste" "F.Mask") (roundrect_rratio 0.25) (net 170 "AI_CH1_IN"))
     (pad "6" smd roundrect (at 2.1 0.325) (size 1.4 0.45) (layers "F.Cu" "F.Paste" "F.Mask") (roundrect_rratio 0.25) (net 63 "ADC1_CH1"))
-    (pad "7" smd roundrect (at 2.1 -0.325) (size 1.4 0.45) (layers "F.Cu" "F.Paste" "F.Mask") (roundrect_rratio 0.25) (net 5 "+3V3A"))
-    (pad "8" smd roundrect (at 2.1 -0.975) (size 1.4 0.45) (layers "F.Cu" "F.Paste" "F.Mask") (roundrect_rratio 0.25) (net 62 "ADC1_CH0"))
+    (pad "7" smd roundrect (at 2.1 -0.325) (size 1.4 0.45) (layers "F.Cu" "F.Paste" "F.Mask") (roundrect_rratio 0.25) (net 63 "ADC1_CH1"))
+    (pad "8" smd roundrect (at 2.1 -0.975) (size 1.4 0.45) (layers "F.Cu" "F.Paste" "F.Mask") (roundrect_rratio 0.25) (net 5 "+3V3A"))
     (fp_rect (start -3.050 -1.800) (end 3.050 1.800) (stroke (width 0.05) (type solid)) (fill none) (layer "F.CrtYd") (uuid "MFG-AI-U20-CY"))
   )
@@
     (property "Value" "1k" (at 0 1.2) (layer "F.Fab") (effects (font (size 0.5 0.5) (thickness 0.08))))
     (pad "1" smd roundrect (at -0.51 0) (size 0.54 0.64) (layers "F.Cu" "F.Paste" "F.Mask") (roundrect_rratio 0.25) (net 119 "AI_CH1_FILT"))
-    (pad "2" smd roundrect (at 0.51 0) (size 0.54 0.64) (layers "F.Cu" "F.Paste" "F.Mask") (roundrect_rratio 0.25) (net 63 "ADC1_CH1"))
+    (pad "2" smd roundrect (at 0.51 0) (size 0.54 0.64) (layers "F.Cu" "F.Paste" "F.Mask") (roundrect_rratio 0.25) (net 170 "AI_CH1_IN"))
     (fp_rect (start -1.030 -0.570) (end 1.030 0.570) (stroke (width 0.05) (type solid)) (fill none) (layer "F.CrtYd") (uuid "MFG-AI-R27-CY"))
   )
@@
     (property "Reference" "C61" (at 0 -1.2) (layer "F.SilkS") (effects (font (size 0.5 0.5) (thickness 0.08))))
     (property "Value" "100nF" (at 0 1.2) (layer "F.Fab") (effects (font (size 0.5 0.5) (thickness 0.08))))
-    (pad "1" smd roundrect (at -0.51 0) (size 0.54 0.64) (layers "F.Cu" "F.Paste" "F.Mask") (roundrect_rratio 0.25) (net 63 "ADC1_CH1"))
+    (pad "1" smd roundrect (at -0.51 0) (size 0.54 0.64) (layers "F.Cu" "F.Paste" "F.Mask") (roundrect_rratio 0.25) (net 170 "AI_CH1_IN"))
     (pad "2" smd roundrect (at 0.51 0) (size 0.54 0.64) (layers "F.Cu" "F.Paste" "F.Mask") (roundrect_rratio 0.25) (net 1 "GND"))
     (fp_rect (start -1.030 -0.570) (end 1.030 0.570) (stroke (width 0.05) (type solid)) (fill none) (layer "F.CrtYd") (uuid "MFG-AI-C61-CY"))
@@
     (property "Value" "1k" (at 0 1.2) (layer "F.Fab") (effects (font (size 0.5 0.5) (thickness 0.08))))
     (pad "1" smd roundrect (at -0.51 0) (size 0.54 0.64) (layers "F.Cu" "F.Paste" "F.Mask") (roundrect_rratio 0.25) (net 120 "AI_CH2_FILT"))
-    (pad "2" smd roundrect (at 0.51 0) (size 0.54 0.64) (layers "F.Cu" "F.Paste" "F.Mask") (roundrect_rratio 0.25) (net 64 "ADC1_CH2"))
+    (pad "2" smd roundrect (at 0.51 0) (size 0.54 0.64) (layers "F.Cu" "F.Paste" "F.Mask") (roundrect_rratio 0.25) (net 171 "AI_CH2_IN"))
     (fp_rect (start -1.030 -0.570) (end 1.030 0.570) (stroke (width 0.05) (type solid)) (fill none) (layer "F.CrtYd") (uuid "MFG-AI-R31-CY"))
   )
@@
     (property "Reference" "C62" (at 0 -1.2) (layer "F.SilkS") (effects (font (size 0.5 0.5) (thickness 0.08))))
     (property "Value" "100nF" (at 0 1.2) (layer "F.Fab") (effects (font (size 0.5 0.5) (thickness 0.08))))
-    (pad "1" smd roundrect (at -0.51 0) (size 0.54 0.64) (layers "F.Cu" "F.Paste" "F.Mask") (roundrect_rratio 0.25) (net 64 "ADC1_CH2"))
+    (pad "1" smd roundrect (at -0.51 0) (size 0.54 0.64) (layers "F.Cu" "F.Paste" "F.Mask") (roundrect_rratio 0.25) (net 171 "AI_CH2_IN"))
     (pad "2" smd roundrect (at 0.51 0) (size 0.54 0.64) (layers "F.Cu" "F.Paste" "F.Mask") (roundrect_rratio 0.25) (net 1 "GND"))
     (fp_rect (start -1.030 -0.570) (end 1.030 0.570) (stroke (width 0.05) (type solid)) (fill none) (layer "F.CrtYd") (uuid "MFG-AI-C62-CY"))
@@
     (property "Value" "1k" (at 0 1.2) (layer "F.Fab") (effects (font (size 0.5 0.5) (thickness 0.08))))
     (pad "1" smd roundrect (at -0.51 0) (size 0.54 0.64) (layers "F.Cu" "F.Paste" "F.Mask") (roundrect_rratio 0.25) (net 121 "AI_CH3_FILT"))
-    (pad "2" smd roundrect (at 0.51 0) (size 0.54 0.64) (layers "F.Cu" "F.Paste" "F.Mask") (roundrect_rratio 0.25) (net 65 "ADC1_CH3"))
+    (pad "2" smd roundrect (at 0.51 0) (size 0.54 0.64) (layers "F.Cu" "F.Paste" "F.Mask") (roundrect_rratio 0.25) (net 172 "AI_CH3_IN"))
     (fp_rect (start -1.030 -0.570) (end 1.030 0.570) (stroke (width 0.05) (type solid)) (fill none) (layer "F.CrtYd") (uuid "MFG-AI-R35-CY"))
   )
@@
     (property "Reference" "C63" (at 0 -1.2) (layer "F.SilkS") (effects (font (size 0.5 0.5) (thickness 0.08))))
     (property "Value" "100nF" (at 0 1.2) (layer "F.Fab") (effects (font (size 0.5 0.5) (thickness 0.08))))
-    (pad "1" smd roundrect (at -0.51 0) (size 0.54 0.64) (layers "F.Cu" "F.Paste" "F.Mask") (roundrect_rratio 0.25) (net 65 "ADC1_CH3"))
+    (pad "1" smd roundrect (at -0.51 0) (size 0.54 0.64) (layers "F.Cu" "F.Paste" "F.Mask") (roundrect_rratio 0.25) (net 172 "AI_CH3_IN"))
     (pad "2" smd roundrect (at 0.51 0) (size 0.54 0.64) (layers "F.Cu" "F.Paste" "F.Mask") (roundrect_rratio 0.25) (net 1 "GND"))
     (fp_rect (start -1.030 -0.570) (end 1.030 0.570) (stroke (width 0.05) (type solid)) (fill none) (layer "F.CrtYd") (uuid "MFG-AI-C63-CY"))
@@
     (pad "1" smd roundrect (at -2.1 -0.975) (size 1.4 0.45) (layers "F.Cu" "F.Paste" "F.Mask") (roundrect_rratio 0.25) (net 64 "ADC1_CH2"))
     (pad "2" smd roundrect (at -2.1 -0.325) (size 1.4 0.45) (layers "F.Cu" "F.Paste" "F.Mask") (roundrect_rratio 0.25) (net 64 "ADC1_CH2"))
-    (pad "3" smd roundrect (at -2.1 0.325) (size 1.4 0.45) (layers "F.Cu" "F.Paste" "F.Mask") (roundrect_rratio 0.25) (net 65 "ADC1_CH3"))
+    (pad "3" smd roundrect (at -2.1 0.325) (size 1.4 0.45) (layers "F.Cu" "F.Paste" "F.Mask") (roundrect_rratio 0.25) (net 171 "AI_CH2_IN"))
     (pad "4" smd roundrect (at -2.1 0.975) (size 1.4 0.45) (layers "F.Cu" "F.Paste" "F.Mask") (roundrect_rratio 0.25) (net 1 "GND"))
-    (pad "5" smd roundrect (at 2.1 0.975) (size 1.4 0.45) (layers "F.Cu" "F.Paste" "F.Mask") (roundrect_rratio 0.25) (net 65 "ADC1_CH3"))
+    (pad "5" smd roundrect (at 2.1 0.975) (size 1.4 0.45) (layers "F.Cu" "F.Paste" "F.Mask") (roundrect_rratio 0.25) (net 172 "AI_CH3_IN"))
     (pad "6" smd roundrect (at 2.1 0.325) (size 1.4 0.45) (layers "F.Cu" "F.Paste" "F.Mask") (roundrect_rratio 0.25) (net 65 "ADC1_CH3"))
-    (pad "7" smd roundrect (at 2.1 -0.325) (size 1.4 0.45) (layers "F.Cu" "F.Paste" "F.Mask") (roundrect_rratio 0.25) (net 5 "+3V3A"))
-    (pad "8" smd roundrect (at 2.1 -0.975) (size 1.4 0.45) (layers "F.Cu" "F.Paste" "F.Mask") (roundrect_rratio 0.25) (net 64 "ADC1_CH2"))
+    (pad "7" smd roundrect (at 2.1 -0.325) (size 1.4 0.45) (layers "F.Cu" "F.Paste" "F.Mask") (roundrect_rratio 0.25) (net 65 "ADC1_CH3"))
+    (pad "8" smd roundrect (at 2.1 -0.975) (size 1.4 0.45) (layers "F.Cu" "F.Paste" "F.Mask") (roundrect_rratio 0.25) (net 5 "+3V3A"))
     (fp_rect (start -3.050 -1.800) (end 3.050 1.800) (stroke (width 0.05) (type solid)) (fill none) (layer "F.CrtYd") (uuid "MFG-AI-U21-CY"))
   )
