File: hardware/kicad/STM32H743_DataLogger/STM32H743_DataLogger.kicad_pcb (KiCad board)
At the start: 4 copper layers, 160 x 100 mm, 6 parts

Commit message: Sync the floorplan sketch to the real layout
STM32H743_DataLogger.kicad_pcb is the human-readable floorplan view, and
it had drifted: it named the Ethernet PHY as LAN8742A when the design uses
a W5500 SPI controller, its block labels still sat at the pre-re-floorplan
positions, and it advertised 0.5mm/0.3mm vias when the board now needs
0.45mm/0.25mm to fan the LQFP-100 out.

Block labels moved onto the regions they actually describe and the missing
ones added: isolated RS485/CAN, the relay bank, storage and the WiFi
module. The terminal-block note now says which field wiring is on which
edge rather than claiming everything is along the bottom.

Co-Authored-By: Claude Opus 5 <noreply@anthropic.com>
Claude-Session: https://claude.ai/code/session_01XsiZ6LJT6X46LKY8yEbRbx
Other:
- board text added: "DIGITAL INPUTS 8ch optocoupled"
- board text added: "ETHERNET W5500 SPI + RJ45"
- board text added: "FIELD TERMINALS: RS485/CAN + DI x8 ON TOP EDGE, 24VDC + AI x4 + DO x4 ON BOTTOM EDGE"
- board text added: "ISOLATED RS485 + CAN (field side, notched pour + milled barrier slots)"
- board text added: "PCB SPECIFICATIONS: Board: 160x100mm, 4-Layer, 1.6mm, FR-4 TG170 Copper: 1oz (35um) all layers Finish: ENIG (Electroless Nickel Immersion Gold) Min Track: 0.15mm (6mil) Min Clearance: 0.125mm (5mil) Min Via: 0.45mm/0.25mm (pad/drill) Impedance: 50ohm single-ended (ETH), controlled Solder Mask: Green, both sides Silkscreen: White, both sides Operating Temp: -40C to +85C (Industrial)"
- board text added: "RELAY OUTPUTS 4ch"
- board text added: "STM32H743VIT6 MCU + Decoupling + Crystal + BLE"
- board text added: "STORAGE microSD + Flash + EEPROM"
- board text added: "WIRELESS LoRa / WiFi / LTE + SIM socket"
- board text added: "WiFi ATWINC1500"
- board text removed: "DIGITAL I/O + RS485 + CAN"
- board text removed: "ETHERNET LAN8742A + RJ45"
- board text removed: "PCB SPECIFICATIONS: Board: 160x100mm, 4-Layer, 1.6mm, FR-4 TG170 Copper: 1oz (35um) all layers Finish: ENIG (Electroless Nickel Immersion Gold) Min Track: 0.15mm (6mil) Min Clearance: 0.15mm (6mil) Min Via: 0.5mm/0.3mm (pad/drill) Impedance: 50ohm single-ended (ETH), controlled Solder Mask: Green, both sides Silkscreen: White, both sides Operating Temp: -40C to +85C (Industrial)"
- board text removed: "STM32H743VIT6 MCU + Decoupling + Crystal"
- board text removed: "TERMINAL BLOCKS (BOTTOM EDGE)"
- board text removed: "WIRELESS LoRa+BLE/WiFi +GSM/LTE"
Changed lines of the file:
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@@
   (gr_rect (start 5 5) (end 45 40)
     (stroke (width 0.15) (type dash)) (fill none) (layer "Dwgs.User") (uuid "PCB-AREA-PSU"))
-  (gr_text "POWER SUPPLY\n24V->5V->3.3V" (at 25 22.5) (layer "Dwgs.User")
+  (gr_text "POWER SUPPLY\n24V->5V->3.3V" (at 39 49) (layer "Dwgs.User")
     (effects (font (size 1.5 1.5) (thickness 0.15)) (justify center))
     (uuid "PCB-TXT-PSU"))
@@
   (gr_rect (start 50 20) (end 110 80)
     (stroke (width 0.15) (type dash)) (fill none) (layer "Dwgs.User") (uuid "PCB-AREA-MCU"))
-  (gr_text "STM32H743VIT6\nMCU + Decoupling\n+ Crystal" (at 80 50) (layer "Dwgs.User")
+  (gr_text "STM32H743VIT6\nMCU + Decoupling\n+ Crystal + BLE" (at 80 47) (layer "Dwgs.User")
     (effects (font (size 1.5 1.5) (thickness 0.15)) (justify center))
     (uuid "PCB-TXT-MCU"))
@@
   (gr_rect (start 120 5) (end 155 40)
     (stroke (width 0.15) (type dash)) (fill none) (layer "Dwgs.User") (uuid "PCB-AREA-ETH"))
-  (gr_text "ETHERNET\nLAN8742A + RJ45" (at 137.5 22.5) (layer "Dwgs.User")
+  (gr_text "ETHERNET\nW5500 SPI + RJ45" (at 133 29) (layer "Dwgs.User")
     (effects (font (size 1.5 1.5) (thickness 0.15)) (justify center))
     (uuid "PCB-TXT-ETH"))
@@
   (gr_rect (start 115 45) (end 155 95)
     (stroke (width 0.15) (type dash)) (fill none) (layer "Dwgs.User") (uuid "PCB-AREA-WL"))
-  (gr_text "WIRELESS\nLoRa+BLE/WiFi\n+GSM/LTE" (at 135 70) (layer "Dwgs.User")
+  (gr_text "WIRELESS\nLoRa / WiFi / LTE\n+ SIM socket" (at 125 55) (layer "Dwgs.User")
     (effects (font (size 1.5 1.5) (thickness 0.15)) (justify center))
     (uuid "PCB-TXT-WL"))
@@
   (gr_rect (start 5 55) (end 45 95)
     (stroke (width 0.15) (type dash)) (fill none) (layer "Dwgs.User") (uuid "PCB-AREA-AI"))
-  (gr_text "ANALOG INPUTS\n4ch 4-20mA/0-10V" (at 25 75) (layer "Dwgs.User")
+  (gr_text "ANALOG INPUTS\n4ch 4-20mA/0-10V" (at 36 84) (layer "Dwgs.User")
     (effects (font (size 1.5 1.5) (thickness 0.15)) (justify center))
     (uuid "PCB-TXT-AI"))
@@
   (gr_rect (start 50 82) (end 110 98)
     (stroke (width 0.15) (type dash)) (fill none) (layer "Dwgs.User") (uuid "PCB-AREA-DIO"))
-  (gr_text "DIGITAL I/O + RS485 + CAN" (at 80 90) (layer "Dwgs.User")
+  (gr_text "DIGITAL INPUTS\n8ch optocoupled" (at 88 26) (layer "Dwgs.User")
     (effects (font (size 1.5 1.5) (thickness 0.15)) (justify center))
     (uuid "PCB-TXT-DIO"))
   ;; Connectors along edges
-  (gr_text "TERMINAL BLOCKS (BOTTOM EDGE)" (at 80 98) (layer "Cmts.User")
+  (gr_text "ISOLATED RS485 + CAN\n(field side, notched pour\n+ milled barrier slots)" (at 33 16) (layer "Dwgs.User")
+    (effects (font (size 1.4 1.4) (thickness 0.15)) (justify center))
+    (uuid "PCB-TXT-FB"))
+  (gr_text "RELAY OUTPUTS 4ch" (at 97 82) (layer "Dwgs.User")
+    (effects (font (size 1.5 1.5) (thickness 0.15)) (justify center))
+    (uuid "PCB-TXT-DO"))
+  (gr_text "STORAGE\nmicroSD + Flash + EEPROM" (at 40 70) (layer "Dwgs.User")
+    (effects (font (size 1.2 1.2) (thickness 0.12)) (justify center))
+    (uuid "PCB-TXT-ST"))
+  (gr_text "WiFi ATWINC1500" (at 26 70) (layer "Dwgs.User")
+    (effects (font (size 1.2 1.2) (thickness 0.12)) (justify center))
+    (uuid "PCB-TXT-WIFI"))
+  (gr_text "FIELD TERMINALS: RS485/CAN + DI x8 ON TOP EDGE, 24VDC + AI x4 + DO x4 ON BOTTOM EDGE" (at 80 99) (layer "Cmts.User")
     (effects (font (size 1 1) (thickness 0.1)) (justify center))
     (uuid "PCB-TXT-CONN"))
@@
   ;; DESIGN RULES TEXT
   ;; ============================================================
-  (gr_text "PCB SPECIFICATIONS:\nBoard: 160x100mm, 4-Layer, 1.6mm, FR-4 TG170\nCopper: 1oz (35um) all layers\nFinish: ENIG (Electroless Nickel Immersion Gold)\nMin Track: 0.15mm (6mil)\nMin Clearance: 0.15mm (6mil)\nMin Via: 0.5mm/0.3mm (pad/drill)\nImpedance: 50ohm single-ended (ETH), controlled\nSolder Mask: Green, both sides\nSilkscreen: White, both sides\nOperating Temp: -40C to +85C (Industrial)"
+  (gr_text "PCB SPECIFICATIONS:\nBoard: 160x100mm, 4-Layer, 1.6mm, FR-4 TG170\nCopper: 1oz (35um) all layers\nFinish: ENIG (Electroless Nickel Immersion Gold)\nMin Track: 0.15mm (6mil)\nMin Clearance: 0.125mm (5mil)\nMin Via: 0.45mm/0.25mm (pad/drill)\nImpedance: 50ohm single-ended (ETH), controlled\nSolder Mask: Green, both sides\nSilkscreen: White, both sides\nOperating Temp: -40C to +85C (Industrial)"
     (at 5 105) (layer "Cmts.User")
     (effects (font (size 1.2 1.2) (thickness 0.12)) (justify left))
