File: hardware/kicad/STM32H743_DataLogger/STM32H743_MCU.kicad_sch (KiCad schematic)
At the start: 35 parts, among them J10 SWD Debug, J11 USB-C, J12 UART Debug Console, J13 BOOT0 Select, J14 TC2050-IDC SWD, U10 STM32H743VIT6, Y1 25MHz, Y2 32.768kHz

Commit message: Complete mfg PCB placement, fix designator conflicts, sync BOM
Manufacturing PCB (STM32H743_DataLogger_mfg.kicad_pcb):
- Add all missing multi-channel footprints: analog channels 1-3
  (D11-D13, R24-R35, C61-C63) plus second op-amp U21
- Add full 8-channel digital input chain (R100-R107 limiters,
  U30/U32-U38 optocouplers, R108-R115 pull-ups) with new
  DI_n_LED nets instead of floating net 0
- Add relays K2-K4 and replace the oversized SANYOU SRD placeholder
  with an HF46F-G/5-HS1T form-A footprint; wire relay contacts to
  J40-J43 via new DOn_NO / DOn_COM nets
- Add C104 (EEPROM decoupling), LED4 + R17 (comm activity indicator)
- Rename the BLE indicator from LED4 to LED5 to match the schematic
- Replace silkscreen branding with the full P9E block (company mark,
  P9E Microsystems Pvt Ltd, www.p9e.in, product, specs) on F.SilkS and
  P/N, S/N, compliance marks and origin on B.SilkS; www.p9e.io and the
  stale "SCADA Systems" text are gone
- Resolve all 26 footprint overlaps, pull the USB-C receptacle fully
  on-board, move fiducials clear of mounting holes, and drop the 22
  stitching vias that landed on pads

Schematics:
- Renumber Digital_IO resistors to R100-R115 and the eighth
  optocoupler to U38, removing the R31x/R40x placeholder designators
  and the R30/R31/R40/R41 collisions with Analog_Inputs and RS485_CAN
- Add C104 to Storage and LED4 + R17 to the MCU sheet

BOM: update the digital I/O and analog designator ranges to match,
add R17, correct the relay type to SPST-NO, and refresh the totals
(116 line items, 211 components).

Co-Authored-By: Claude Opus 5 <noreply@anthropic.com>
Claude-Session: https://claude.ai/code/session_01XsiZ6LJT6X46LKY8yEbRbx
Parts:
- added LED4: Orange COMM, LED_SMD:LED_0603_1608Metric, symbol Device:LED
- added R17: 1k, Resistor_SMD:R_0402_1005Metric, symbol Device:R
Changed lines of the file:
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@@
     (property "Manufacturer" "Yageo" (at 228.6 168.275 0) (effects (font (size 1.27 1.27)) hide))
+  )
+  ;; LED4 - communication activity (PD15), R17 current limit
+  (symbol (lib_id "Device:LED") (at 241.3 158.75) (unit 1)
+    (exclude_from_sim no) (in_bom yes) (on_board yes) (dnp no)
+    (uuid "MCU-0084-LED4")
+    (property "Reference" "LED4" (at 241.3 153.67 0) (effects (font (size 1.27 1.27))))
+    (property "Value" "Orange COMM" (at 241.3 156.21 0) (effects (font (size 1.27 1.27))))
+    (property "Footprint" "LED_SMD:LED_0603_1608Metric" (at 241.3 158.75 0) (effects (font (size 1.27 1.27)) hide))
+    (property "MPN" "19-213/Y2C-CQ2R2L/3T" (at 241.3 158.75 0) (effects (font (size 1.27 1.27)) hide))
+    (property "Manufacturer" "Everlight" (at 241.3 158.75 0) (effects (font (size 1.27 1.27)) hide))
+  )
+  (symbol (lib_id "Device:R") (at 241.3 168.275) (unit 1)
+    (exclude_from_sim no) (in_bom yes) (on_board yes) (dnp no)
+    (uuid "MCU-0085-R17")
+    (property "Reference" "R17" (at 243.84 168.275 0) (effects (font (size 1.27 1.27))))
+    (property "Value" "1k" (at 241.3 170.815 0) (effects (font (size 1.27 1.27))))
+    (property "Footprint" "Resistor_SMD:R_0402_1005Metric" (at 241.3 168.275 0) (effects (font (size 1.27 1.27)) hide))
+    (property "MPN" "RC0402FR-071KL" (at 241.3 168.275 0) (effects (font (size 1.27 1.27)) hide))
+    (property "Manufacturer" "Yageo" (at 241.3 168.275 0) (effects (font (size 1.27 1.27)) hide))
   )
   ;; ============================================================

Commit message: Close six unconnected nets found while exporting the netlist
Exporting the board to Specctra for routing surfaced six nets with only
one pad on them — they had nothing to connect to:

- VBUCK_BST reached only U1 pin 1. The buck had no bootstrap capacitor,
  so the high-side switch could never turn on and the 24V-to-5V stage
  would not start. Added C11 (100nF) from BST to the SW node.
- USART1_TX_BUF and USART1_RX_BUF dead-ended at R14/R15. J12 tapped the
  MCU side of the 33R series resistors, so the debug header was wired
  straight to the MCU and the resistors sat in mid-air. J12 now taps the
  buffered side, putting them in circuit as intended.
- GSM_DTR, GSM_RI and LORA_DIO1 reached only their module pins. The MCU
  has no spare pad (all 100 are assigned), so DTR gets a 10k pull-down
  (R18) to hold the modem out of sleep rather than floating, and RI and
  DIO1 come out to probe pads TP9/TP10.

Also added TP1-TP8 to the schematics; they existed only as PCB pads, so
the netlist and the board disagreed about them.

BOM now 120 line items / 219 components. Placement re-verified: 227
footprints, zero courtyard collisions, nothing off-board.

Co-Authored-By: Claude Opus 5 <noreply@anthropic.com>
Claude-Session: https://claude.ai/code/session_01XsiZ6LJT6X46LKY8yEbRbx
Parts:
- added TP5: SWDIO, TestPoint:TestPoint_Pad_1.0x1.0mm, symbol Connector:TestPoint
- added TP6: SWCLK, TestPoint:TestPoint_Pad_1.0x1.0mm, symbol Connector:TestPoint
- added TP7: NRST, TestPoint:TestPoint_Pad_1.0x1.0mm, symbol Connector:TestPoint
- added TP8: BOOT0, TestPoint:TestPoint_Pad_1.0x1.0mm, symbol Connector:TestPoint
Changed lines of the file:
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@@
   ;; PIN ASSIGNMENTS (documented as text annotation)
   ;; ============================================================
-  (text "STM32H743VIT6 PIN ASSIGNMENTS (Rev 1.2 - SPI-based architecture):\n\n=== COMMUNICATION PERIPHERALS ===\nSPI1/LoRa SX1276: PA5(SCK), PA6(MISO), PB5(MOSI), PA4(NSS_LORA), PC13(DIO0_IRQ), PC2(RST)\nSPI2/WiFi ATWINC1500: PB13(SCK), PB14(MISO), PB15(MOSI), PB12(NSS_WIFI), PB1(CHIP_EN), PC0(RST_N), PD10(IRQ_N)\nSPI3/Flash W25Q64JV: PB3(SCK), PB4(MISO), PB2(MOSI), PA15(NSS_FLASH) [REMAPPED from PC10-12 for SDMMC1]\nSPI4/Ethernet W5500: PE2(SCK), PE5(MISO), PE6(MOSI), PE4(NSS_ETH), PE3(RST_N), PB0(INT_N)\nUSART1/Debug Console: PA9(TX), PA10(RX) -> J12 header (115200 baud)\nUART4/GSM SIM7600: PA0(TX), PC11(RX), PC3(PWR_KEY), PD11(STATUS)\nUART7/BLE RN4870: PE8(TX), PE7(RX), PD12(RST_N_BLE), PD13(STATUS_BLE)\nFDCAN1: PD0(RX), PD1(TX)\nUSART2/RS485: PD5(TX), PD6(RX), PD4(DE/RE)\n\n=== STORAGE ===\nSDMMC1 (4-bit): PC8(D0), PC9(D1), PC10(D2), PC11(D3), PC12(CLK), PD2(CMD)\nI2C1/EEPROM: PB6(SCL), PB7(SDA)\n\n=== ANALOG / DIGITAL I/O ===\nADC1: PA0-PA3 (4 channels, 16-bit)\nDI GPIO: PD3, PD7, PE0, PE1, PE9-PE12 (8x digital inputs via optocouplers)\nDO GPIO: PE13-PE15, PD14 (4x relay driver outputs)\n\n=== SYSTEM ===\nUSB_OTG_FS: PA11(DM), PA12(DP)\nSWD: PA13(SWDIO), PA14(SWCLK)\nBOOT0: Dedicated pin, jumper J13 (GND=flash boot, 3V3=DFU mode), R16 10k pull-down default\nNRST: Reset with RC filter + TPS3823 WDT output\nHSE: PH0(OSC_IN), PH1(OSC_OUT) - 25MHz\nLSE: PC14(OSC32_IN), PC15(OSC32_OUT) - 32.768kHz\nWDT_KICK: PB8 (TPS3823 WDI input)\n\n=== PROGRAMMING INTERFACES ===\nJ10: 10-pin ARM SWD header (Samtec FTSH-105-01-L-DV-K, 1.27mm pitch)\nJ11: USB-C connector (USB_OTG_FS for DFU programming)\nJ12: UART debug console header (4-pin 2.54mm: VCC/TX/RX/GND, USART1 PA9/PA10)\nJ13: BOOT0 select jumper (3-pin: GND-BOOT0-3V3, default=flash boot)\nJ14: Tag-Connect TC2050-IDC pads (production programming, same SWD signals as J10)\n\nNOTE: RMII pins freed (PA1,PA2,PA7,PB11,PC1,PC4,PC5) by using W5500 SPI Ethernet\nNOTE: SPI3 remapped from PC10-12 to PB3/PB4/PB2 to free PC8-12 for SDMMC1 4-bit SD card"
+  (text "STM32H743VIT6 PIN ASSIGNMENTS (Rev 1.2 - SPI-based architecture):\n\n=== COMMUNICATION PERIPHERALS ===\nSPI1/LoRa SX1276: PA5(SCK), PA6(MISO), PB5(MOSI), PA4(NSS_LORA), PC13(DIO0_IRQ), PC2(RST)\nSPI2/WiFi ATWINC1500: PB13(SCK), PB14(MISO), PB15(MOSI), PB12(NSS_WIFI), PB1(CHIP_EN), PC0(RST_N), PD10(IRQ_N)\nSPI3/Flash W25Q64JV: PB3(SCK), PB4(MISO), PB2(MOSI), PA15(NSS_FLASH) [REMAPPED from PC10-12 for SDMMC1]\nSPI4/Ethernet W5500: PE2(SCK), PE5(MISO), PE6(MOSI), PE4(NSS_ETH), PE3(RST_N), PB0(INT_N)\nUSART1/Debug Console: PA9(TX), PA10(RX) -> J12 header (115200 baud)\nUART4/GSM SIM7600: PA0(TX), PC11(RX), PC3(PWR_KEY), PD11(STATUS)\nUART7/BLE RN4870: PE8(TX), PE7(RX), PD12(RST_N_BLE), PD13(STATUS_BLE)\nFDCAN1: PD0(RX), PD1(TX)\nUSART2/RS485: PD5(TX), PD6(RX), PD4(DE/RE)\n\n=== STORAGE ===\nSDMMC1 (4-bit): PC8(D0), PC9(D1), PC10(D2), PC11(D3), PC12(CLK), PD2(CMD)\nI2C1/EEPROM: PB6(SCL), PB7(SDA)\n\n=== ANALOG / DIGITAL I/O ===\nADC1: PA0-PA3 (4 channels, 16-bit)\nDI GPIO: PD3, PD7, PE0, PE1, PE9-PE12 (8x digital inputs via optocouplers)\nDO GPIO: PE13-PE15, PD14 (4x relay driver outputs)\n\n=== SYSTEM ===\nUSB_OTG_FS: PA11(DM), PA12(DP)\nSWD: PA13(SWDIO), PA14(SWCLK)\nBOOT0: Dedicated pin, jumper J13 (GND=flash boot, 3V3=DFU mode), R16 10k pull-down default\nNRST: Reset with RC filter + TPS3823 WDT output\nHSE: PH0(OSC_IN), PH1(OSC_OUT) - 25MHz\nLSE: PC14(OSC32_IN), PC15(OSC32_OUT) - 32.768kHz\nWDT_KICK: PB8 (TPS3823 WDI input)\n\n=== PROGRAMMING INTERFACES ===\nJ10: 10-pin ARM SWD header (Samtec FTSH-105-01-L-DV-K, 1.27mm pitch)\nJ11: USB-C connector (USB_OTG_FS for DFU programming)\nJ12: UART debug console header (4-pin 2.54mm: VCC/TX/RX/GND) - wired to the\n     BUFFERED side of R14/R15, i.e. USART1_TX_BUF / USART1_RX_BUF, so the 33R\n     series resistors are actually in circuit\nJ13: BOOT0 select jumper (3-pin: GND-BOOT0-3V3, default=flash boot)\nJ14: Tag-Connect TC2050-IDC pads (production programming, same SWD signals as J10)\n\nNOTE: RMII pins freed (PA1,PA2,PA7,PB11,PC1,PC4,PC5) by using W5500 SPI Ethernet\nNOTE: SPI3 remapped from PC10-12 to PB3/PB4/PB2 to free PC8-12 for SDMMC1 4-bit SD card"
     (exclude_from_sim no)
     (at 25.4 25.4 0)
@@
     (uuid "MCU-TEXT-0001")
   )
+  ;; Probe test points
+  (symbol (lib_id "Connector:TestPoint") (at 165.1 190.5) (unit 1)
+    (exclude_from_sim no) (in_bom yes) (on_board yes) (dnp no)
+    (uuid "MCU-0090-TP5")
+    (property "Reference" "TP5" (at 165.1 186.69 0) (effects (font (size 1.27 1.27))))
+    (property "Value" "SWDIO" (at 165.1 189.23 0) (effects (font (size 1.27 1.27))))
+    (property "Footprint" "TestPoint:TestPoint_Pad_1.0x1.0mm" (at 165.1 190.5 0) (effects (font (size 1.27 1.27)) hide))
+  )
+  (symbol (lib_id "Connector:TestPoint") (at 177.8 190.5) (unit 1)
+    (exclude_from_sim no) (in_bom yes) (on_board yes) (dnp no)
+    (uuid "MCU-0091-TP6")
+    (property "Reference" "TP6" (at 177.8 186.69 0) (effects (font (size 1.27 1.27))))
+    (property "Value" "SWCLK" (at 177.8 189.23 0) (effects (font (size 1.27 1.27))))
+    (property "Footprint" "TestPoint:TestPoint_Pad_1.0x1.0mm" (at 177.8 190.5 0) (effects (font (size 1.27 1.27)) hide))
+  )
+  (symbol (lib_id "Connector:TestPoint") (at 190.5 190.5) (unit 1)
+    (exclude_from_sim no) (in_bom yes) (on_board yes) (dnp no)
+    (uuid "MCU-0092-TP7")
+    (property "Reference" "TP7" (at 190.5 186.69 0) (effects (font (size 1.27 1.27))))
+    (property "Value" "NRST" (at 190.5 189.23 0) (effects (font (size 1.27 1.27))))
+    (property "Footprint" "TestPoint:TestPoint_Pad_1.0x1.0mm" (at 190.5 190.5 0) (effects (font (size 1.27 1.27)) hide))
+  )
+  (symbol (lib_id "Connector:TestPoint") (at 203.2 190.5) (unit 1)
+    (exclude_from_sim no) (in_bom yes) (on_board yes) (dnp no)
+    (uuid "MCU-0093-TP8")
+    (property "Reference" "TP8" (at 203.2 186.69 0) (effects (font (size 1.27 1.27))))
+    (property "Value" "BOOT0" (at 203.2 189.23 0) (effects (font (size 1.27 1.27))))
+    (property "Footprint" "TestPoint:TestPoint_Pad_1.0x1.0mm" (at 203.2 190.5 0) (effects (font (size 1.27 1.27)) hide))
+  )
 )
